File: OSSIComms/OSSIComms/OSSIComms.sch (EAGLE design)
At the start: 174 parts, among them Q2 NX-3215, U1 MAX890L, U10 LMZ10503EXT, U11 OPA347, U12 TPS73233, U14 RF5110G, U15 HSWA2-30DR+, U16 MAX2640, U2 ADF7021-N, U3 ADF7021-N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

Commit message: OSSI COMMS PA components value changed based on Swisscube
Parts:
- C92: value 10nF -> 10pF
- C93: value 330pF -> 15pF
- L11: value 2.7nH -> 3.9nH
- L12: value 6.8nH -> 1.5nH
- L5: value 1uH 3012 -> 39nH 3012, 1A rating
- R35: value 0 -> 330nH
- R36: value 18 -> 11nH
Changed lines of the file:
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@@
 <part name="GND66" library="OSSI" deviceset="GND" device=""/>
 <part name="GND67" library="OSSI" deviceset="GND" device=""/>
-<part name="L11" library="OSSI" deviceset="L" device="0603(1608)" value="2.7nH"/>
+<part name="L11" library="OSSI" deviceset="L" device="0603(1608)" value="3.9nH"/>
 <part name="C81" library="OSSI" deviceset="C" device="0603(1608)" value="47pF"/>
 <part name="C82" library="OSSI" deviceset="C" device="0603(1608)" value="1nF"/>
@@
 <part name="C89" library="OSSI" deviceset="C" device="0603(1608)" value="10nF"/>
 <part name="GND78" library="OSSI" deviceset="GND" device=""/>
-<part name="L12" library="OSSI" deviceset="L" device="0603(1608)" value="6.8nH"/>
-<part name="R35" library="OSSI" deviceset="R" device="0603(1608)" value="0"/>
+<part name="L12" library="OSSI" deviceset="L" device="0603(1608)" value="1.5nH"/>
+<part name="R35" library="OSSI" deviceset="R" device="0603(1608)" value="330nH"/>
 <part name="C90" library="OSSI" deviceset="C" device="1210(3225)-TMK325" value="3.3uF"/>
 <part name="C91" library="OSSI" deviceset="C" device="0603(1608)" value="1nF"/>
-<part name="C92" library="OSSI" deviceset="C" device="0603(1608)" value="10nF"/>
+<part name="C92" library="OSSI" deviceset="C" device="0603(1608)" value="10pF"/>
 <part name="GND79" library="OSSI" deviceset="GND" device=""/>
 <part name="GND80" library="OSSI" deviceset="GND" device=""/>
 <part name="GND81" library="OSSI" deviceset="GND" device=""/>
-<part name="C93" library="OSSI" deviceset="C" device="0603(1608)" value="330pF"/>
+<part name="C93" library="OSSI" deviceset="C" device="0603(1608)" value="15pF"/>
 <part name="GND82" library="OSSI" deviceset="GND" device=""/>
-<part name="R36" library="OSSI" deviceset="R" device="0603(1608)" value="18"/>
+<part name="R36" library="OSSI" deviceset="R" device="0603(1608)" value="11nH"/>
 <part name="C94" library="OSSI" deviceset="C" device="0603(1608)" value="330pF"/>
 <part name="C95" library="OSSI" deviceset="C" device="0603(1608)" value="1nF"/>
 <part name="C96" library="OSSI" deviceset="C" device="0603(1608)" value="10nF"/>
 <part name="GND73" library="OSSI" deviceset="GND" device=""/>
-<part name="L5" library="OSSI" deviceset="L" device="NR3012" value="1uH 3012"/>
+<part name="L5" library="OSSI" deviceset="L" device="NR3012" value="39nH 3012, 1A rating"/>
 <part name="X2" library="OSSI" deviceset="JTAG10PINMINI" device="-H"/>
 <part name="3.3VCOMMS9" library="OSSI" deviceset="3.3VCOMMS" device=""/>
