File: OSSIComms/OSSIComms/OSSIComms.brd (EAGLE design)
At the start: 94 x 94 mm, 174 parts, among them Q2 NX-3215, U1 MAX890L, U10 LMZ10503EXT, U11 OPA347, U12 TPS73233, U14 RF5110G, U15 HSWA2-30DR+, U16 MAX2640, U2 ADF7021-N, U3 ADF7021-N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

Commit message: OSSI COMMS PA components value changed based on Swisscube
Parts:
- C92: value 10nF -> 10pF
- C93: value 330pF -> 15pF
- L11: value 2.7nH -> 3.9nH
- L12: value 6.8nH -> 1.5nH
- L5: value 1uH 3012 -> 39nH 3012, 1A rating
- R35: value 0 -> 330nH
- R36: value 18 -> 11nH
Changed lines of the file:
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@@
 <attribute name="VALUE" x="48.03775" y="16.79575" size="1.27" layer="27" rot="R180"/>
 </element>
-<element name="L11" library="OSSI" package="L0603(1608)" value="2.7nH" x="33.02" y="14.605" smashed="yes" rot="R180">
+<element name="L11" library="OSSI" package="L0603(1608)" value="3.9nH" x="33.02" y="14.605" smashed="yes" rot="R180">
 <attribute name="NAME" x="35.814" y="17.2085" size="1.27" layer="25" font="vector" rot="R180"/>
 <attribute name="VALUE" x="33.909" y="16.637" size="1.27" layer="27" rot="R180"/>
@@
 <attribute name="VALUE" x="44.73575" y="8.9535" size="1.27" layer="27" rot="R90"/>
 </element>
-<element name="L12" library="OSSI" package="L0603(1608)" value="6.8nH" x="41.91" y="18.7325" smashed="yes" rot="R270">
+<element name="L12" library="OSSI" package="L0603(1608)" value="1.5nH" x="41.91" y="18.7325" smashed="yes" rot="R270">
 <attribute name="NAME" x="42.926" y="18.3515" size="1.27" layer="25" font="vector"/>
 <attribute name="VALUE" x="39.878" y="19.6215" size="1.27" layer="27" rot="R270"/>
 </element>
-<element name="R35" library="OSSI" package="R0603(1608)" value="0" x="41.91" y="21.74875" smashed="yes" rot="R270">
+<element name="R35" library="OSSI" package="R0603(1608)" value="330nH" x="41.91" y="21.74875" smashed="yes" rot="R270">
 <attribute name="NAME" x="43.40225" y="21.844" size="1.27" layer="25" font="vector"/>
 <attribute name="VALUE" x="39.878" y="22.63775" size="1.27" layer="27" rot="R270"/>
@@
 <attribute name="VALUE" x="42.164" y="26.32075" size="1.27" layer="27" rot="R180"/>
 </element>
-<element name="C92" library="OSSI" package="C0603(1608)" value="10nF" x="41.275" y="26.3525" smashed="yes" rot="R180">
+<element name="C92" library="OSSI" package="C0603(1608)" value="10pF" x="41.275" y="26.3525" smashed="yes" rot="R180">
 <attribute name="NAME" x="38.6715" y="26.7335" size="1.27" layer="25" font="vector" rot="R180"/>
 <attribute name="VALUE" x="42.164" y="28.3845" size="1.27" layer="27" rot="R180"/>
 </element>
-<element name="C93" library="OSSI" package="C0603(1608)" value="330pF" x="39.52875" y="20.32" smashed="yes" rot="R180">
+<element name="C93" library="OSSI" package="C0603(1608)" value="15pF" x="39.52875" y="20.32" smashed="yes" rot="R180">
 <attribute name="NAME" x="37.87775" y="20.701" size="1.27" layer="25" font="vector" rot="R180"/>
 <attribute name="VALUE" x="40.41775" y="22.352" size="1.27" layer="27" rot="R180"/>
 </element>
-<element name="R36" library="OSSI" package="R0603(1608)" value="18" x="44.60875" y="11.58875" smashed="yes" rot="R270">
+<element name="R36" library="OSSI" package="R0603(1608)" value="11nH" x="44.60875" y="11.58875" smashed="yes" rot="R270">
 <attribute name="NAME" x="45.62475" y="10.89025" size="1.27" layer="25" font="vector"/>
 <attribute name="VALUE" x="42.57675" y="12.47775" size="1.27" layer="27" rot="R270"/>
@@
 <attribute name="VALUE" x="40.8305" y="6.9215" size="1.27" layer="27" rot="R270"/>
 </element>
-<element name="L5" library="OSSI" package="NR3012" value="1uH 3012" x="37.1475" y="13.335" smashed="yes" rot="R270">
+<element name="L5" library="OSSI" package="NR3012" value="39nH 3012, 1A rating" x="37.1475" y="13.335" smashed="yes" rot="R270">
 <attribute name="NAME" x="36.195" y="14.605" size="1.27" layer="25" font="vector" rot="R270"/>
 <attribute name="VALUE" x="33.3375" y="16.51" size="1.27" layer="27" rot="R270"/>
