File: OSSITestBoard/OSSIDevBoard/OSSIDevBoard.sch (EAGLE design)
At the start: 0 parts

Commit message: OSSI Dev Board Alpha added
Parts:
- added C36: (no value), OSSI:C0805(2012)
- added CHASSIS1, CHASSIS2, CHASSIS3: CHASSIS_T_B, OSSI:CHASSIS_T_B
- added H1, H2, H3, H4, H5, H6, H7, H8: MOUNT-PAD-ROUND3.2, OSSI:MOUNT-PAD-ROUND3.2
- added JP1, JP2: (no value), OSSI:JP1Q
- added R39: 511k, OSSI:R0805(2012)
- added SHIELD1: SHIELD_OBC, OSSI:SHIELD_OBC
- added SHIELD2: SHIELD_COMMS, OSSI:SHIELD_COMMS
- added SHIELD3: SHIELD_EPS, OSSI:SHIELD_EPS
- added TP1, TP2, TP3, TP4: TP, OSSI:TP
- added X1, X2: ESQ-126-38-G-D, OSSI:ESQ-126-38-G-D
- added X3, X4, X5: BANANA_PLUG, OSSI:BANANA_PLUG
Connections:
- new net 3.3VOBC: SHIELD1.45, SHIELD1.46, SHIELD2.45, SHIELD2.46, SHIELD3.45, SHIELD3.46, X1.45, X1.46, X2.45, X2.46
- new net ANT_DEPLOY1: SHIELD1.19, SHIELD2.19, SHIELD3.19, X1.19, X2.19
- new net ANT_DEPLOY2: SHIELD1.20, SHIELD2.20, SHIELD3.20, X1.20, X2.20
- new net BAT_-CHRG: SHIELD1.42, SHIELD2.42, SHIELD3.42, X1.42, X2.42
- new net BAT_-FAULT: SHIELD1.44, SHIELD2.44, SHIELD3.44, X1.44, X2.44
- new net BAT_-ON: SHIELD1.38, SHIELD2.38, SHIELD3.38, X1.38, X2.38
- new net BEACON_-FAULT: SHIELD1.30, SHIELD2.30, SHIELD3.30, X1.30, X2.30
- new net BEACON_OFF: SHIELD1.24, SHIELD2.24, SHIELD3.24, X1.24, X2.24
- new net BEACON_SCL: SHIELD1.37, SHIELD2.37, SHIELD3.37, X1.37, X2.37
- new net BEACON_SDA: SHIELD1.39, SHIELD2.39, SHIELD3.39, X1.39, X2.39
- new net COMMS_-FAULT: SHIELD1.32, SHIELD2.32, SHIELD3.32, X1.32, X2.32
- new net COMMS_OFF: SHIELD1.25, SHIELD2.25, SHIELD3.25, X1.25, X2.25
- new net COMMS_SCL: SHIELD1.41, SHIELD2.41, SHIELD3.41, X1.41, X2.41
- new net COMMS_SDA: SHIELD1.43, SHIELD2.43, SHIELD3.43, X1.43, X2.43
- new net GND: SHIELD1.1, SHIELD1.2, SHIELD1.51, SHIELD1.52, SHIELD2.1, SHIELD2.2, SHIELD2.51, SHIELD2.52, SHIELD3.1, SHIELD3.2, SHIELD3.51, SHIELD3.52, TP1.TP, TP2.TP, TP3.TP, TP4.TP, X1.1, X1.2, X1.51, X1.52, X2.1, X2.2, X2.51, X2.52, X4.A
- new net LED_-FAULT: SHIELD1.28, SHIELD2.28, SHIELD3.28, X1.28, X2.28
- new net LED_OFF: SHIELD1.23, SHIELD2.23, SHIELD3.23, X1.23, X2.23
- new net LED_SCL: SHIELD1.33, SHIELD2.33, SHIELD3.33, X1.33, X2.33
- new net LED_SDA: SHIELD1.35, SHIELD2.35, SHIELD3.35, X1.35, X2.35
- new net N$1: JP1.2, SHIELD1.10, SHIELD1.7, SHIELD1.8, SHIELD1.9
- new net N$2: JP2.2, SHIELD2.10, SHIELD2.7, SHIELD2.8, SHIELD2.9
- new net OBC_-FAULT: SHIELD1.34, SHIELD2.34, SHIELD3.34, X1.34, X2.34
- new net OBC_OFF: SHIELD1.26, SHIELD2.26, SHIELD3.26, X1.26, X2.26
- new net PANELTEMP_SCL: SHIELD1.29, SHIELD2.29, SHIELD3.29, X1.29, X2.29
- new net PANELTEMP_SDA: SHIELD1.31, SHIELD2.31, SHIELD3.31, X1.31, X2.31
- new net SCCHG_EN: SHIELD1.21, SHIELD2.21, SHIELD3.21, X1.21, X2.21
- new net SCOUT_-PG: SHIELD1.50, SHIELD2.50, SHIELD3.50, X1.50, X2.50
- new net SCOUT_EN: SHIELD1.22, SHIELD2.22, SHIELD3.22, X1.22, X2.22
- new net SC_-ON: SHIELD1.40, SHIELD2.40, SHIELD3.40, X1.40, X2.40
- new net SC_-PFO: SHIELD1.48, SHIELD2.48, SHIELD3.48, X1.48, X2.48
- new net SECONDARY_SCL: SHIELD1.47, SHIELD2.47, SHIELD3.47, X1.47, X2.47
- new net SECONDARY_SDA: SHIELD1.49, SHIELD2.49, SHIELD3.49, X1.49, X2.49
- new net SOLAR_-ON: SHIELD1.36, SHIELD2.36, SHIELD3.36, X1.36, X2.36
- new net SOLAR_CS1: SHIELD1.15, SHIELD2.15, SHIELD3.15, X1.15, X2.15
- new net SOLAR_CS2: SHIELD1.14, SHIELD2.14, SHIELD3.14, X1.14, X2.14
- new net SOLAR_CS3: SHIELD1.17, SHIELD2.17, SHIELD3.17, X1.17, X2.17
- new net SOLAR_CS4: SHIELD1.16, SHIELD2.16, SHIELD3.16, X1.16, X2.16
- new net SOLAR_CS5: SHIELD1.18, SHIELD2.18, SHIELD3.18, X1.18, X2.18
- new net STRUT_GND: C36.2, CHASSIS1.A, CHASSIS1.B, CHASSIS2.A, CHASSIS2.B, CHASSIS3.A, CHASSIS3.B, H1.MOUNT, H2.MOUNT, H3.MOUNT, H4.MOUNT, H5.MOUNT, H6.MOUNT, H7.MOUNT, H8.MOUNT, R39.1
- new net STRUT_GND1: C36.1, R39.2, SHIELD3.A
- new net SUN: SHIELD1.27, SHIELD2.27, SHIELD3.27, X1.27, X2.27
- new net VBAT: SHIELD1.11, SHIELD1.12, SHIELD2.11, SHIELD2.12, SHIELD3.11, SHIELD3.12, X1.11, X1.12, X2.11, X2.12
- new net VBUS: JP1.1, JP2.1, SHIELD3.10, SHIELD3.7, SHIELD3.8, SHIELD3.9, X1.10, X1.7, X1.8, X1.9, X2.10, X2.7, X2.8, X2.9, X5.A
- new net VSOLAR: SHIELD1.5, SHIELD1.6, SHIELD2.5, SHIELD2.6, SHIELD3.5, SHIELD3.6, X1.5, X1.6, X2.5, X2.6, X3.A
- new net VSUPERCAP: SHIELD1.13, SHIELD2.13, SHIELD3.13, X1.13, X2.13
