File: OSSITestBoard/OSSIDevBoard/OSSIDevBoard.brd (EAGLE design)
At the start: 362 x 130 mm, 27 parts, among them X1 ESQ-126-38-G-D, X2 ESQ-126-38-G-D, X3 BANANA_PLUG, X4 BANANA_PLUG, X5 BANANA_PLUG

Commit message: all values for tuned results are updated
Other:
- board text added: "BAT_TEMP"
- board text added: "BUS_CS"
- board text added: "SC_TEMP"
- board text removed: "SC_PG"
- board text removed: "SUN"
Changed lines of the file:
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@@
 <grid distance="1" unitdist="mm" unit="mm" style="lines" multiple="1" display="yes" altdistance="0.5" altunitdist="mm" altunit="mm"/>
 <layers>
-<layer number="1" name="Top" color="4" fill="1" visible="yes" active="yes"/>
+<layer number="1" name="Top" color="4" fill="1" visible="no" active="yes"/>
 <layer number="2" name="Route2" color="1" fill="3" visible="no" active="no"/>
 <layer number="3" name="Route3" color="4" fill="3" visible="no" active="no"/>
@@
 <layer number="14" name="Route14" color="1" fill="6" visible="no" active="no"/>
 <layer number="15" name="Route15" color="4" fill="6" visible="no" active="no"/>
-<layer number="16" name="Bottom" color="1" fill="1" visible="yes" active="yes"/>
-<layer number="17" name="Pads" color="2" fill="1" visible="yes" active="yes"/>
-<layer number="18" name="Vias" color="2" fill="1" visible="yes" active="yes"/>
-<layer number="19" name="Unrouted" color="6" fill="1" visible="yes" active="yes"/>
-<layer number="20" name="Dimension" color="15" fill="1" visible="yes" active="yes"/>
+<layer number="16" name="Bottom" color="1" fill="1" visible="no" active="yes"/>
+<layer number="17" name="Pads" color="2" fill="1" visible="no" active="yes"/>
+<layer number="18" name="Vias" color="2" fill="1" visible="no" active="yes"/>
+<layer number="19" name="Unrouted" color="6" fill="1" visible="no" active="yes"/>
+<layer number="20" name="Dimension" color="15" fill="1" visible="no" active="yes"/>
 <layer number="21" name="tPlace" color="7" fill="1" visible="yes" active="yes"/>
 <layer number="22" name="bPlace" color="7" fill="1" visible="yes" active="yes"/>
-<layer number="23" name="tOrigins" color="15" fill="1" visible="yes" active="yes"/>
-<layer number="24" name="bOrigins" color="15" fill="1" visible="yes" active="yes"/>
+<layer number="23" name="tOrigins" color="15" fill="1" visible="no" active="yes"/>
+<layer number="24" name="bOrigins" color="15" fill="1" visible="no" active="yes"/>
 <layer number="25" name="tNames" color="7" fill="1" visible="yes" active="yes"/>
 <layer number="26" name="bNames" color="7" fill="1" visible="yes" active="yes"/>
@@
 <text x="356" y="43.5" size="1.27" layer="21" font="vector">L_OFF</text>
 <text x="356" y="46" size="1.27" layer="21" font="vector">C_OFF</text>
-<text x="356" y="48.5" size="1.27" layer="21" font="vector">SUN</text>
+<text x="356" y="48.5" size="1.27" layer="21" font="vector">BUS_CS</text>
 <text x="356" y="51" size="1.27" layer="21" font="vector">T_SCL</text>
 <text x="356" y="53.5" size="1.27" layer="21" font="vector">T_SDA</text>
@@
 <text x="356" y="66.5" size="1.27" layer="21" font="vector">C_SCL</text>
 <text x="356" y="69" size="1.27" layer="21" font="vector">C_SDA</text>
-<text x="356" y="71" size="1.27" layer="21" font="vector">3.3VOBC</text>
+<text x="356" y="71.5" size="1.27" layer="21" font="vector">3.3VOBC</text>
 <text x="344" y="23" size="1.27" layer="21" font="vector">VBUS</text>
 <text x="344" y="25.5" size="1.27" layer="21" font="vector">VBUS</text>
@@
 <text x="341" y="71.5" size="1.27" layer="21" font="vector">3.3VOBC</text>
 <text x="341.5" y="74" size="1.27" layer="21" font="vector">SC_PFO</text>
-<text x="343" y="76.5" size="1.27" layer="21" font="vector">SC_PG</text>
 <text x="345" y="79" size="1.27" layer="21" font="vector">GND</text>
+<text x="344" y="18" size="1.27" layer="21" font="vector">VSOL</text>
+<text x="356" y="18" size="1.27" layer="21" font="vector">VSOL</text>
+<text x="356" y="74" size="1.27" layer="21" font="vector">BAT_TEMP</text>
+<text x="356" y="76.5" size="1.27" layer="21" font="vector">SC_TEMP</text>
 </plain>
 <attributes>
