File: OSSILEDController/OSSILEDController2132/OSSILEDController2132.brd (EAGLE design)
At the start: 70 x 38 mm, 60 parts, among them J1 JTAG-SBW-6, Q1 NX-3215, U1 OPA2347, U12 TPS73233, U2 MSP430F2132, U3 LM7321, U4 MAX1682, U5 MAX890L, U6 MAX4376, U7 TPS3838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

Commit message: MCP1700 SO23 added
Parts:
- removed C34, C35: 1uF 0805, OSSI:C0805(2012)
- removed U12: TPS73233, OSSI:SOT23-5DBV
- added C11, C12: 10uF, LDO Tantal 16V, OSSI:C1206(3216)-A
- added R23: 0, OSSI:R0603(1608)
- added U8: MCP1700_SOT23, OSSI:SOT23
- moved R22 229.7 mm to (39.4, 29.2)
- moved C10 216.8 mm to (38.7, 25.4), flipped to the bottom, turned to 180 degrees
- moved U6 212.3 mm to (39.4, 28.6), flipped to the bottom
- moved R21 199.0 mm to (12.7, 24.1), turned to 270 degrees
- moved R20 195.0 mm to (10.2, 24.1), turned to 270 degrees
- moved R19 193.9 mm to (11.4, 26.7), turned to 180 degrees
- moved C9 191.7 mm to (17.8, 30.5), turned to 180 degrees
- moved C8 190.0 mm to (21.6, 34.3), turned to 270 degrees
- moved U4 181.9 mm to (19.1, 34.3)
- moved U3 165.2 mm to (17.8, 25.4), turned to 270 degrees
- moved C6 165.1 mm to (16.5, 34.3), turned to 270 degrees
- moved R17 114.3 mm to (25.4, 24.1), turned to 270 degrees
- moved R16 107.6 mm to (22.9, 24.1), turned to 270 degrees
- moved R15 104.1 mm to (24.1, 26.7), turned to 180 degrees
- moved C5 102.6 mm to (-27.9, -22.9), turned to 270 degrees
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Connections:
- removed net LED_-RST: U7.3
- new net N$12: C11.2, R23.1
- net 3.3VLED: now also C11.1, U8.2; no longer C34.1, U12.5
- net GND: now also C12.2, R23.2, U8.1; no longer C34.2, C35.2, U12.2
- net N$5: now also C12.1, U8.3; no longer C35.1, U12.1, U12.3
Routing:
- removed copper zone on layer 1, net GND
- removed copper zone on layer 16, net GND
- removed copper zone on layer 1, net LED-
- removed copper zone on layer 16, net LED-
- removed copper zone on layer 16, net N$18
- removed copper zone on layer 1, net VSUPERCAP
