File: OSSILEDController/OSSILEDController2132/OSSILEDController2132.sch (EAGLE design)
At the start: 60 parts, among them J1 JTAG-SBW-6, Q1 NX-3215, U1 OPA2347, U12 TPS73233, U2 MSP430F2132, U3 LM7321, U4 MAX1682, U5 MAX890L, U6 MAX4376, U7 TPS3838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

Commit message: MCP1700 SO23 added
Parts:
- removed C34, C35: 1uF 0805, OSSI:C0805(2012)
- removed U12: TPS73233, OSSI:TPS73233
- added C11, C12: 10uF, LDO Tantal 16V, OSSI:C-TANTAL-A
- added R23: 0, OSSI:R0603(1608)
- added U8: MCP1700_SOT23, OSSI:MCP1700_SOT23
Connections:
- removed net LED_-RST: U7.P$3
- new net N$12: C11.-, R23.1
- net 3.3VLED: now also C11.+, U8.2; no longer C34.1, U12.5
- net GND: now also C12.-, R23.2, U8.1; no longer C34.2, C35.2, U12.2
- net N$5: now also C12.+, U8.3; no longer C35.1, U12.1, U12.3
Other:
- note added: "TEST POINTS!!!!"
Changed lines of the file:
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@@
 <part name="U7" library="OSSI" deviceset="TPS3838" device=""/>
 <part name="GND8" library="OSSI" deviceset="GND" device=""/>
-<part name="U12" library="OSSI" deviceset="TPS732*" device="" technology="33"/>
 <part name="GND9" library="OSSI" deviceset="GND" device=""/>
 <part name="R2" library="OSSI" deviceset="R" device="0603(1608)" value="100k"/>
-<part name="C34" library="OSSI" deviceset="C" device="0805(2012)" value="1uF 0805"/>
-<part name="C35" library="OSSI" deviceset="C" device="0805(2012)" value="1uF 0805"/>
 <part name="GND63" library="OSSI" deviceset="GND" device=""/>
 <part name="3.3VLED6" library="OSSI" deviceset="3.3VLED" device=""/>
@@
 <part name="C10" library="OSSI" deviceset="C" device="0603(1608)" value="100nF"/>
 <part name="R22" library="OSSI" deviceset="R" device="WSR2" value="0.005, 2W RSENSE"/>
+<part name="C11" library="OSSI" deviceset="C-TANTAL-A" device="" value="10uF, LDO Tantal 16V"/>
+<part name="C12" library="OSSI" deviceset="C-TANTAL-A" device="" value="10uF, LDO Tantal 16V"/>
+<part name="R23" library="OSSI" deviceset="R" device="0603(1608)" value="0"/>
+<part name="U8" library="OSSI" deviceset="MCP1700" device="_SOT23"/>
 </parts>
 <sheets>
@@
 <text x="175.26" y="129.54" size="1.778" layer="94">Conntect Test Pin to JTAG!!</text>
 <text x="12.7" y="106.68" size="1.778" layer="94">Check Supercap voltage!!!!!</text>
+<text x="160.02" y="238.76" size="6.4516" layer="94">TEST POINTS!!!!</text>
 </plain>
 <instances>
@@
 <instance part="C3" gate="G$1" x="104.14" y="185.42"/>
 <instance part="U7" gate="G$1" x="167.64" y="185.42"/>
-<instance part="GND8" gate="1" x="119.38" y="172.72"/>
-<instance part="U12" gate="G$1" x="134.62" y="190.5"/>
+<instance part="GND8" gate="1" x="114.3" y="172.72"/>
 <instance part="GND9" gate="1" x="154.94" y="182.88"/>
 <instance part="R2" gate="G$1" x="180.34" y="187.96" rot="R90"/>
-<instance part="C34" gate="G$1" x="152.4" y="185.42"/>
-<instance part="C35" gate="G$1" x="114.3" y="185.42"/>
-<instance part="GND63" gate="1" x="152.4" y="175.26"/>
+<instance part="GND63" gate="1" x="152.4" y="157.48"/>
 <instance part="3.3VLED6" gate="G$1" x="152.4" y="200.66"/>
 <instance part="R7" gate="G$1" x="307.34" y="134.62" rot="R270"/>
@@
 <instance part="C10" gate="G$1" x="347.98" y="149.86" rot="R90"/>
 <instance part="R22" gate="G$1" x="317.5" y="144.78" rot="R270"/>
+<instance part="C11" gate="G$1" x="152.4" y="182.88"/>
+<instance part="C12" gate="G$1" x="114.3" y="185.42"/>
+<instance part="R23" gate="G$1" x="152.4" y="170.18" rot="R270"/>
+<instance part="U8" gate="G$1" x="132.08" y="195.58" rot="R180"/>
 </instances>
 <busses>
@@
 <wire x1="147.32" y1="195.58" x2="152.4" y2="195.58" width="0.1524" layer="91"/>
 <wire x1="152.4" y1="195.58" x2="152.4" y2="200.66" width="0.1524" layer="91"/>
-<pinref part="U12" gate="G$1" pin="5"/>
 <wire x1="152.4" y1="195.58" x2="177.8" y2="195.58" width="0.1524" layer="91"/>
 <wire x1="177.8" y1="195.58" x2="177.8" y2="190.5" width="0.1524" layer="91"/>
@@
 <wire x1="180.34" y1="195.58" x2="180.34" y2="193.04" width="0.1524" layer="91"/>
 <junction x="177.8" y="195.58"/>
-<pinref part="C34" gate="G$1" pin="1"/>
 <wire x1="152.4" y1="187.96" x2="152.4" y2="195.58" width="0.1524" layer="91"/>
 <pinref part="3.3VLED6" gate="G$1" pin="3.3VLED"/>
+<pinref part="C11" gate="G$1" pin="+"/>
+<wire x1="152.4" y1="185.42" x2="152.4" y2="187.96" width="0.1524" layer="91"/>
+<pinref part="U8" gate="G$1" pin="2"/>
+<wire x1="142.24" y1="198.12" x2="144.78" y2="198.12" width="0.1524" layer="91"/>
+<wire x1="144.78" y1="198.12" x2="144.78" y2="195.58" width="0.1524" layer="91"/>
+<wire x1="144.78" y1="195.58" x2="147.32" y2="195.58" width="0.1524" layer="91"/>
 </segment>
 <segment>
@@
 </segment>
 <segment>
+<pinref part="C12" gate="G$1" pin="-"/>
+<wire x1="114.3" y1="180.34" x2="114.3" y2="177.8" width="0.1524" layer="91"/>
 <pinref part="GND8" gate="1" pin="GND"/>
-<wire x1="119.38" y1="175.26" x2="119.38" y2="177.8" width="0.1524" layer="91"/>
-<wire x1="119.38" y1="177.8" x2="119.38" y2="190.5" width="0.1524" layer="91"/>
-<wire x1="119.38" y1="190.5" x2="124.46" y2="190.5" width="0.1524" layer="91"/>
-<pinref part="U12" gate="G$1" pin="2"/>
-<pinref part="C35" gate="G$1" pin="2"/>
-<wire x1="114.3" y1="180.34" x2="114.3" y2="177.8" width="0.1524" layer="91"/>
-<wire x1="114.3" y1="177.8" x2="119.38" y2="177.8" width="0.1524" layer="91"/>
-<junction x="119.38" y="177.8"/>
+<wire x1="114.3" y1="175.26" x2="114.3" y2="177.8" width="0.1524" layer="91"/>
 </segment>
 <segment>
@@
 <wire x1="160.02" y1="185.42" x2="154.94" y2="185.42" width="0.1524" layer="91"/>
 <junction x="154.94" y="185.42"/>
-</segment>
-<segment>
-<pinref part="GND63" gate="1" pin="GND"/>
-<pinref part="C34" gate="G$1" pin="2"/>
-<wire x1="152.4" y1="177.8" x2="152.4" y2="180.34" width="0.1524" layer="91"/>
 </segment>
 <segment>
@@
 <wire x1="358.14" y1="149.86" x2="358.14" y2="144.78" width="0.1524" layer="91"/>
 <junction x="358.14" y="144.78"/>
+</segment>
+<segment>
+<pinref part="GND63" gate="1" pin="GND"/>
+<pinref part="R23" gate="G$1" pin="2"/>
+<wire x1="152.4" y1="160.02" x2="152.4" y2="162.56" width="0.1524" layer="91"/>
+<pinref part="U8" gate="G$1" pin="1"/>
+<wire x1="152.4" y1="162.56" x2="152.4" y2="165.1" width="0.1524" layer="91"/>
+<wire x1="142.24" y1="193.04" x2="144.78" y2="193.04" width="0.1524" layer="91"/>
+<wire x1="144.78" y1="193.04" x2="144.78" y2="162.56" width="0.1524" layer="91"/>
+<wire x1="144.78" y1="162.56" x2="152.4" y2="162.56" width="0.1524" layer="91"/>
+<junction x="152.4" y="162.56"/>
 </segment>
 </net>
@@
 <wire x1="104.14" y1="187.96" x2="104.14" y2="195.58" width="0.1524" layer="91"/>
 <junction x="104.14" y="195.58"/>
-<pinref part="U12" gate="G$1" pin="1"/>
-<pinref part="U12" gate="G$1" pin="3"/>
 <wire x1="121.92" y1="195.58" x2="124.46" y2="195.58" width="0.1524" layer="91"/>
-<wire x1="124.46" y1="185.42" x2="121.92" y2="185.42" width="0.1524" layer="91"/>
-<wire x1="121.92" y1="185.42" x2="121.92" y2="195.58" width="0.1524" layer="91"/>
-<junction x="121.92" y="195.58"/>
 <wire x1="104.14" y1="195.58" x2="114.3" y2="195.58" width="0.1524" layer="91"/>
-<pinref part="C35" gate="G$1" pin="1"/>
 <wire x1="114.3" y1="195.58" x2="121.92" y2="195.58" width="0.1524" layer="91"/>
 <wire x1="114.3" y1="187.96" x2="114.3" y2="195.58" width="0.1524" layer="91"/>
 <junction x="114.3" y="195.58"/>
+<pinref part="C12" gate="G$1" pin="+"/>
+<pinref part="U8" gate="G$1" pin="3"/>
 </segment>
 </net>
@@
 <wire x1="60.96" y1="38.1" x2="60.96" y2="43.18" width="0.1524" layer="91"/>
 <label x="60.96" y="43.18" size="1.778" layer="95" rot="R90" xref="yes"/>
-</segment>
-</net>
-<net name="LED_-RST" class="0">
-<segment>
-<pinref part="U7" gate="G$1" pin="P$3"/>
-<wire x1="160.02" y1="180.34" x2="157.48" y2="180.34" width="0.1524" layer="91"/>
-<wire x1="157.48" y1="180.34" x2="157.48" y2="154.94" width="0.1524" layer="91"/>
-<label x="157.48" y="154.94" size="1.778" layer="95" rot="R180" xref="yes"/>
 </segment>
 </net>
@@
 </segment>
 </net>
+<net name="N$12" class="0">
+<segment>
+<pinref part="R23" gate="G$1" pin="1"/>
+<pinref part="C11" gate="G$1" pin="-"/>
+<wire x1="152.4" y1="175.26" x2="152.4" y2="177.8" width="0.1524" layer="91"/>
+</segment>
+</net>
