File: OSSIEPS/OSSIEPS/OSSIEPS.sch (EAGLE design)
At the start: 138 parts, among them U1 LT3479, U10 LTC4411, U11 SN74LVC1T45-EP, U12 SN74LVC1T45-EP, U13 MAX890L, U14 MAX890L, U2 LT3479, U3 LT3652, U4 LTC4411, U5 LTC4411, U6 LTC4425, U7 TPS63020, U8 LTC4411, U9 LTC4411, X1 ESQ-126-38-G-D, X10 P-PAD-S, X11 P-PAD-S, X12 P-PAD-S, X13 P-PAD-S, X14 P-PAD-S, X15 P-PAD-S, X16 P-PAD-S, X17 P-PAD-S, X18 P-PAD-S, X2 DF13DF13-8P-1.25DSA, X3 DF13DF13-8P-1.25DSA, X4 DF13-10P-1.25DSA, X5 P-PAD, X6 P-PAD, X7 P-PAD, X8 E62-10K, X9 P-PAD-S

Commit message: EPS comment added to Chassis Structure GND move
Other:
- note added: "Move this to front !!!!"
Changed lines of the file:
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@@
 <sheet>
 <plain>
+<text x="58.42" y="50.8" size="1.778" layer="94">Move this to front !!!!</text>
 </plain>
 <instances>

Commit message: Chage EPS StrutGND R size to 1206!!! note added
Other:
- note added: "Chage Resistor Size to 1206!!!"
Changed lines of the file:
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@@
 <plain>
 <text x="58.42" y="50.8" size="1.778" layer="94">Move this to front !!!!</text>
+<text x="48.26" y="81.28" size="1.778" layer="94">Chage Resistor Size to 1206!!!</text>
 </plain>
 <instances>
