File: OSSIComms/OSSICommsBeaconNewNew/OSSIBeaconNewNew.sch (EAGLE design)
At the start: 116 parts, among them Q1 NX-3215, U1 MAX890L, U10 MSP430F2132, U2 ADL5530, U3 NC7SZ04, U4 ADF7012, U5 OPA2347, U6 MAX890L, U7 MAX6369, U8 MCP1700_SOT23, U9 TPS3838, X1 ESQ-126-38-G-D, X2 RFCON-MCX-R/A, X3 5268-02, X4 JTAG10PINMINI-H, X5 5268-03, X7 P-PAD-S, X8 P-PAD-S

Commit message: schematics renumbered
Parts:
- removed R39: 511, OSSI:RWSL1206
- added R36: 100k, OSSI:R0603(1608)
- C1: value 10nF -> (none); device OSSI:C0603(1608) -> OSSI:C0805(2012)
- C10: value 10nF -> 100nF
- C11: value 1nF -> 22pF
- C12: value DNP -> 22pF
- C13: value 2.2uF, 0805 -> 22pF; device OSSI:C0805(2012) -> OSSI:C0603(1608)
- C14: value 100pF -> 1nF
- C15: value 1uF,0603 -> 10nF
- C16: value 68pF -> 1nF
- C17: value 1000pF -> 2.2uF, 0805; device OSSI:C0603(1608) -> OSSI:C0805(2012)
- C18: value 1uF 0805 -> 100pF; device OSSI:C0805(2012) -> OSSI:C0603(1608)
- C19: value 22pF -> 1uF
- C2: value 1uF -> 10nF
- C20: value 22nF -> (none)
- C21: value 100pF -> DNP
- C22: value 1nF -> 100pF
- C23: value 1uF -> 1uF 0805; device OSSI:C0603(1608) -> OSSI:C0805(2012)
- C24: value 22pF -> 1uF,0603
- C25: value (none) -> 22nF
- C26: value 22pF -> 68pF
- C27: value 22pF -> 1000pF
- C28: value TBD -> 22pF
- C29: value TBD -> 100nF
- C3: value 100nF -> 10nF
- C30, C33: value 100nF -> TBD
- C31: value 1uF -> 100nF
- C32: value 100nF -> 12.5pF
- C34: value 10uF, LDO Tantal 16V -> 12.5pF; device OSSI:C-TANTAL-A -> OSSI:C0603(1608)
- C35: value 10uF, LDO Tantal 16V -> 100nF; device OSSI:C-TANTAL-A -> OSSI:C0603(1608)
- C36: value 12.5pF -> 100nF
- C37: value 12.5pF -> 1uF
- C39: value 100nF -> 10uF, LDO Tantal 16V; device OSSI:C0603(1608) -> OSSI:C-TANTAL-A
- C4: value 10nF -> (none)
- C40: value 10nF -> 10uF, LDO Tantal 16V; device OSSI:C0603(1608) -> OSSI:C-TANTAL-A
- C41: value 22uF,1210 -> 10nF; device OSSI:C1210(3225)-GCM32 -> OSSI:C0603(1608)
- C42: value 100nF -> 22uF,1210; device OSSI:C0603(1608) -> OSSI:C1210(3225)-GCM32
- C43: value (none) -> 100nF; device OSSI:C0805(2012) -> OSSI:C0603(1608)
- C9: value (none) -> 1uF
- L2: value 10nH -> 68nH
- L3: value 470nH, 1008 size -> 68nH; device OSSI:L1008(2502) -> OSSI:L0603(1608)
- L4: value 68nH -> 10nH
- L5: value 68nH -> 470nH, 1008 size; device OSSI:L0603(1608) -> OSSI:L1008(2502)
- R1: value 100k -> 511; device OSSI:R0603(1608) -> OSSI:RWSL1206
- R10: value 100k -> 5.1k
- R11: value 100k -> 47k
- R12, R22: value 100k -> 4.7k
- R13: value 100k -> 250
- R14: value 100k -> 10k
- R15: value 23.7k -> 1k
- R16: value 0 -> 250
- R17: value 10k -> 100k
- R19, R20: value 250 -> 4.7k
- R21, R29, R30, R35: value 4.7k -> 100k
- R23: value 1k -> 4.7k
- R24: value 47k -> 4.7k
- R3: value 100k -> 6.2k
- R33: value 4.7k -> 0
- R34: value 4.7k -> 23.7k
- R4: value 6.2k -> 100k
- R5: value 1M -> 100k
- R6: value 2.4k -> 0
- R7: value 5.1k -> 1M
- R9: value 0 -> 2.4k
- U1: value MAX890L -> ADL5530; device OSSI:MAX890L -> OSSI:ADL5530
- U10: value MSP430F2132 -> MCP1700_SOT23; device OSSI:MSP430F2132 -> OSSI:MCP1700_SOT23
- U2: value ADL5530 -> MAX890L; device OSSI:ADL5530 -> OSSI:MAX890L
- U5: value OPA2347 -> MAX6369; device OSSI:OPA2347 -> OSSI:MAX6369
- U6: value MAX890L -> MSP430F2132; device OSSI:MAX890L -> OSSI:MSP430F2132
- U7: value MAX6369 -> OPA2347; device OSSI:MAX6369 -> OSSI:OPA2347
- U8: value MCP1700_SOT23 -> TPS3838; device OSSI:MCP1700_SOT23 -> OSSI:TPS3838
- U9: value TPS3838 -> MAX890L; device OSSI:TPS3838 -> OSSI:MAX890L
- X1: value ESQ-126-38-G-D -> P-PAD-S; device OSSI:ESQ-126-38-G-D -> OSSI:P-PAD-S
- X2: value RFCON-MCX-R/A -> ESQ-126-38-G-D; device OSSI:RFCON-MCX-R/A -> OSSI:ESQ-126-38-G-D
- X3: value 5268-02 -> P-PAD-S; device OSSI:5268-02 -> OSSI:P-PAD-S
- X4: value JTAG10PINMINI-H -> RFCON-MCX-R/A; device OSSI:JTAG10PINMINI-H -> OSSI:RFCON-MCX-R/A
- X5: value 5268-03 -> 5268-02; device OSSI:5268-03 -> OSSI:5268-02
- X7: value P-PAD-S -> 5268-03; device OSSI:P-PAD-S -> OSSI:5268-03
- X8: value P-PAD-S -> JTAG10PINMINI-H; device OSSI:P-PAD-S -> OSSI:JTAG10PINMINI-H
Connections:
- net 3.3VBEACON: now also C35.1, C36.1, C40.+, C42.1, R14.2, R36.2, R5.2, U5.P$4, U5.P$5, U5.P$6, U5.P$8, U6.2, U7A.V+, U8.P$5, X5.1, X8.4; no longer C30.1, C35.+, C38.1, C40.1, R17.2, R22.2, R3.2, U5A.V+, U7.P$4, U7.P$5, U7.P$6, U7.P$8, U8.2, U9.P$5, X3.1, X4.4
- net 3.3VOBC: now also X2.45, X2.46; no longer X1.45, X1.46
- net ADC0: now also U6.8, U7B.-IN, U7B.OUT; no longer U10.8, U5B.-IN, U5B.OUT
- net ADC1: now also U6.9, U7A.-IN, U7A.OUT; no longer U10.9, U5A.-IN, U5A.OUT
- net ANT_DEPLOY1: now also X2.19; no longer X1.19
- net ANT_DEPLOY2: now also X2.20; no longer X1.20
- net BAT_-CHRG: now also X2.42; no longer X1.42
- net BAT_-FAULT: now also X2.44; no longer X1.44
- net BAT_-ON: now also X2.38; no longer X1.38
- net BAT_TEMP: now also X2.47; no longer X1.47
- net BEACON_-FAULT: now also U9.P$8, X2.30; no longer U6.P$8, X1.30
- net BEACON_CE: now also R22.2; no longer R26.2
- net BEACON_CWCONTROL: now also R11.1, R12.2, X5.2; no longer R24.1, R25.2, X3.2
- net BEACON_DATA: now also R28.2; no longer R32.2
- net BEACON_MUXOUT: now also R26.2; no longer R30.2
- net BEACON_OFF: now also C37.1, R35.2, U9.P$3, X2.24; no longer C31.1, R14.2, U6.P$3, X1.24
- net BEACON_RFOUT: now also C13.2, C2.1, L3.2; no longer C1.1, C27.2, L5.2
- net BEACON_SCL: now also R13.1, R14.1, X2.37; no longer R17.1, R20.1, X1.37
- net BEACON_SCLK: now also R25.2; no longer R29.2
- net BEACON_SDA: now also R16.1, X2.39; no longer R19.1, X1.39
- net BEACON_SDATA: now also R24.2; no longer R28.2
- net BEACON_SLE: now also R23.2; no longer R27.2
- net BEACON_TXCLK: now also R27.2; no longer R31.2
- net BEACON_WDT_RST: now also C31.1, U5.P$7, U8.P$3; no longer C33.1, U7.P$7, U9.P$3
- net BUS_CS: now also R30.1, X2.27; no longer R13.1, X1.27
- net COMMS_-FAULT: now also X2.32; no longer X1.32
- net COMMS_OFF: now also X2.25; no longer X1.25
- net COMMS_SCL: now also X2.41; no longer X1.41
- net COMMS_SDA: now also X2.43; no longer X1.43
- net GND: now also C1.2, C11.1, C12.1, C17.1, C18.2, C20.2, C22.2, C23.1, C24.2, C34.2, C35.2, C39.-, C9.2, R11.2, R17.2, R2.1, R29.2, R3.1, R32.2, R33.2, R34.1, R35.1, R9.2, U1.1, U1.3, U1.4, U1.5, U1.6, U1.8, U10.1, U2.P$4, U5.P$2, U6.4, U7A.V-, U8.P$1, U8.P$2, U9.P$4, X1.P$1, X2.1, X2.51, X2.52, X4.2, X4.3, X4.4, X4.5, X7.1, X8.9; no longer C14.2, C16.1, C18.1, C2.2, C21.2, C23.2, C24.1, C25.2, C27.1, C3.2, C34.-, C39.2, C40.2, R10.2, R12.2, R14.1, R15.1, R16.2, R21.2, R24.2, R39.1, R4.1, R6.2, U1.P$4, U10.4, U2.1, U2.3, U2.4, U2.5, U2.6, U2.8, U5A.V-, U6.P$4, U7.P$2, U8.1, U9.P$1, U9.P$2, X1.1, X1.2, X1.51, X1.52, X2.3, X2.4, X2.5, X4.9, X5.1, X8.P$1
- net LED_-FAULT: now also X2.28; no longer X1.28
- net LED_OFF: now also X2.23; no longer X1.23
- net LED_SCL: now also X2.33; no longer X1.33
- net LED_SDA: now also X2.35; no longer X1.35
- net N$1: now also R15.1, U6.11; no longer R23.1, U10.11
- net N$10: now also R13.2, U6.13; no longer R20.2, U10.13
- net N$11: now also R20.2, U6.16; no longer R34.2, U10.16
- net N$12: now also U5.P$1, U6.10; no longer U10.10, U7.P$1
- net N$13: now also C29.1, R12.1, U6.14; no longer C39.1, R25.1, U10.14
- net N$14: now also L4.1; no longer L2.1
- net N$15: now also L4.2; no longer L2.2
- net N$16: now also C23.2, C25.1; no longer C18.2, C20.1
- net N$17: now also C25.2; no longer C20.2
- net N$19: now also C9.1, R4.1, U2.P$3; no longer C2.1, R2.1, U1.P$3
- net N$2: now also U6.27, X8.3; no longer U10.27, X4.3
- net N$20: now also C27.1, R9.1; no longer C17.1, R6.1
- net N$21: now also R3.2, U2.P$5; no longer R4.2, U1.P$5
- net N$22: now also C30.1, R17.1, R21.2, U7B.+IN; no longer C28.1, R10.1, R11.2, U5B.+IN
- net N$23: now also C14.2, L5.2; no longer C22.2, L3.2
- net N$24: now also C28.1, R10.1; no longer C19.1, R7.1
- net N$25: now also C17.2; no longer C13.2
- net N$26: now also C26.2, C27.2, R10.2; no longer C16.2, C17.2, R7.2
- net N$27: now also C18.1, C19.1, L5.1, R6.2; no longer C21.1, C23.1, L3.1, R9.2
- net N$28: now also C2.2, U1.2; no longer C1.2, U2.2
- net N$29: now also C11.2, C14.1, L2.1; no longer C22.1, C24.2, L4.1
- net N$3: now also U6.26, X8.5; no longer U10.26, X4.5
- net N$30: now also C3.1, U1.7; no longer C4.1, U2.7
- net N$31: now also R31.1, X8.10; no longer R35.1, X4.10
- net N$32: now also R34.2, U9.P$5; no longer R15.2, U6.P$5
- net N$33: now also C33.1, R29.1, R30.2, U7A.+IN; no longer C29.1, R12.1, R13.2, U5A.+IN
- net N$34: now also C3.2; no longer C4.2
- net N$35: now also C4.1; no longer C9.1
- net N$36: now also C12.2, L2.2, L3.1; no longer C26.2, L4.2, L5.1
- net N$37: now also C4.2, X4.1; no longer C9.2, X2.1
- net N$38: now also C16.2, C21.1, R7.2; no longer C11.2, C12.1, R5.2
- net N$39: now also R19.2, U6.15; no longer R33.2, U10.15
- net N$4: now also U6.25, X8.7; no longer U10.25, X4.7
- net N$40: now also C40.-, R33.1; no longer C35.-, R16.1
- net N$41: now also R28.1, U6.24; no longer R32.1, U10.24
- net N$42: now also R27.1, U6.23; no longer R31.1, U10.23
- net N$43: now also R26.1, U6.22; no longer R30.1, U10.22
- net N$44: now also R25.1, U6.21; no longer R29.1, U10.21
- net N$45: now also R24.1, U6.20; no longer R28.1, U10.20
- net N$46: now also R23.1, U6.19; no longer R27.1, U10.19
- net N$47: now also R22.1, U6.18; no longer R26.1, U10.18
- net N$5: now also C34.1, U6.5; no longer C37.1, U10.5
- net N$6: now also C32.1, U6.6; no longer C36.1, U10.6
- net N$666: now also C38.1, C39.+, U10.3, U9.P$6, U9.P$7; no longer C32.1, C34.+, U6.P$6, U6.P$7, U8.3
- net N$69: now also C16.1; no longer C11.1
- net N$7: now also R15.2; no longer R23.2
- net N$8: now also U6.28, X8.1; no longer U10.28, X4.1
- net N$9: now also R16.2, U6.12; no longer R19.2, U10.12
- net OBC_-FAULT: now also X2.34; no longer X1.34
- net OBC_OFF: now also X2.26; no longer X1.26
- net OSC1: now also C21.2; no longer C12.2
- net OSC2: now also R7.1; no longer R5.1
- net PANELTEMP_SCL: now also X2.29; no longer X1.29
- net PANELTEMP_SDA: now also X2.31; no longer X1.31
- net PA_-FAULT: now also R5.1, U2.P$8, U6.3; no longer R3.1, U1.P$8, U10.3
- net PA_ON: now also R2.2, U6.17; no longer R1.2, U10.17
- net RESETBEACON: now also R31.2, R36.1, U6.7, U8.P$4; no longer R22.1, R35.2, U10.7, U9.P$4
- net RXD: now also R20.1, X7.3; no longer R34.1, X5.3
- net SCCHG_EN: now also X2.21; no longer X1.21
- net SCOUT_-PG: now also X2.50; no longer X1.50
- net SCOUT_EN: now also X2.22; no longer X1.22
- net SC_-ON: now also X2.40; no longer X1.40
- net SC_-PFO: now also X2.48; no longer X1.48
- net SOLAR_-ON: now also X2.36; no longer X1.36
- net SOLAR_CS1: now also X2.15; no longer X1.15
- net SOLAR_CS2: now also X2.14; no longer X1.14
- net SOLAR_CS3: now also X2.17; no longer X1.17
- net SOLAR_CS4: now also X2.16; no longer X1.16
- net SOLAR_CS5: now also X2.18; no longer X1.18
- net STRUT_GND: now also C1.1, R1.2; no longer C43.1, R39.2
- net SUPERCAP_TEMP: now also X2.49; no longer X1.49
- net TEST: now also R32.1, U6.1, X8.8; no longer R21.1, U10.1, X4.8
- net TXD: now also R19.1, X7.2; no longer R33.1, X5.2
- net VBAT: now also X2.11, X2.12; no longer X1.11, X1.12
- net VBEACON_PA: now also C10.1, U2.P$6, U2.P$7; no longer C3.1, U1.P$6, U1.P$7
- net VBUS: now also R21.1, R4.2, U2.P$1, U2.P$2, U9.P$1, U9.P$2, X2.10, X2.7, X2.8, X2.9, X3.P$1; no longer R11.1, R2.2, U1.P$1, U1.P$2, U6.P$1, U6.P$2, X1.10, X1.7, X1.8, X1.9, X7.P$1
- net VCCRF: now also C20.1, C22.1, C24.1, C43.1, R6.1; no longer C10.1, C14.1, C25.1, C42.1, R9.1
- net VSOLAR: now also X2.3, X2.4, X2.5, X2.6; no longer X1.3, X1.4, X1.5, X1.6
- net VSUPERCAP: now also X2.13; no longer X1.13
Other:
- moved on the sheet: C11, C12, C13, C14, C15, C16, C17, C18, C19, C2, C20, C21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

Commit message: beacon valued corrected
Parts:
- C12: value 22pF -> 39pF
- C20: value (none) -> 1uF,0603 Too Small!!
- C4: value (none) -> 10nF
- L6: value 5~15R ferrite bead -> 7 R Ferrite Bead, 3A
- R29: value 100k -> DNP
- R30: value 100k -> 10k
- R32: value 4.7k -> 100k
Changed lines of the file:
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@@
 <part name="3.3VBEACON4" library="OSSI" deviceset="3.3VBEACON" device=""/>
 <part name="GND10" library="OSSI" deviceset="GND" device=""/>
-<part name="R29" library="OSSI" deviceset="R" device="0603(1608)" value="100k"/>
+<part name="R29" library="OSSI" deviceset="R" device="0603(1608)" value="DNP"/>
 <part name="R17" library="OSSI" deviceset="R" device="0603(1608)" value="100k"/>
 <part name="C33" library="OSSI" deviceset="C" device="0603(1608)" value="TBD"/>
@@
 <part name="C36" library="OSSI" deviceset="C" device="0603(1608)" value="100nF"/>
 <part name="GND19" library="OSSI" deviceset="GND" device=""/>
-<part name="R30" library="OSSI" deviceset="R" device="0603(1608)" value="100k"/>
+<part name="R30" library="OSSI" deviceset="R" device="0603(1608)" value="10k"/>
 <part name="R21" library="OSSI" deviceset="R" device="0603(1608)" value="100k"/>
 <part name="U9" library="OSSI" deviceset="MAX890L" device=""/>
@@
 <part name="C18" library="OSSI" deviceset="C" device="0603(1608)" value="100pF"/>
 <part name="GND22" library="OSSI" deviceset="GND" device=""/>
-<part name="C20" library="OSSI" deviceset="C" device="0603(1608)"/>
+<part name="C20" library="OSSI" deviceset="C" device="0603(1608)" value="1uF,0603 Too Small!!"/>
 <part name="GND23" library="OSSI" deviceset="GND" device=""/>
 <part name="C24" library="OSSI" deviceset="C" device="0603(1608)" value="1uF,0603"/>
@@
 <part name="L3" library="OSSI" deviceset="L" device="0603(1608)" value="68nH"/>
 <part name="C11" library="OSSI" deviceset="C" device="0603(1608)" value="22pF"/>
-<part name="C12" library="OSSI" deviceset="C" device="0603(1608)" value="22pF"/>
+<part name="C12" library="OSSI" deviceset="C" device="0603(1608)" value="39pF"/>
 <part name="C13" library="OSSI" deviceset="C" device="0603(1608)" value="22pF"/>
 <part name="GND30" library="OSSI" deviceset="GND" device=""/>
@@
 <part name="GND32" library="OSSI" deviceset="GND" device=""/>
 <part name="F1" library="OSSI" deviceset="LFCN-160" device=""/>
-<part name="C4" library="OSSI" deviceset="C" device="0603(1608)"/>
+<part name="C4" library="OSSI" deviceset="C" device="0603(1608)" value="10nF"/>
 <part name="GND33" library="OSSI" deviceset="GND" device=""/>
 <part name="GND34" library="OSSI" deviceset="GND" device=""/>
 <part name="3.3VOBC3" library="OSSI" deviceset="3.3VBEACON" device=""/>
 <part name="VCCRF3" library="OSSI" deviceset="VCCRF" device=""/>
-<part name="L6" library="OSSI" deviceset="L" device="0805(2012)" value="5~15R ferrite bead"/>
+<part name="L6" library="OSSI" deviceset="L" device="0805(2012)" value="7 R Ferrite Bead, 3A"/>
 <part name="C41" library="OSSI" deviceset="C" device="0603(1608)" value="10nF"/>
 <part name="C43" library="OSSI" deviceset="C" device="0603(1608)" value="100nF"/>
@@
 <part name="VSOLAR4" library="OSSI" deviceset="VSOLAR" device=""/>
 <part name="STRUT_GND1" library="OSSI" deviceset="STRUT_GND" device=""/>
-<part name="R32" library="OSSI" deviceset="R" device="0603(1608)" value="4.7k"/>
+<part name="R32" library="OSSI" deviceset="R" device="0603(1608)" value="100k"/>
 <part name="GND36" library="OSSI" deviceset="GND" device=""/>
 <part name="X7" library="OSSI" deviceset="5268-03" device=""/>

Commit message: beacon value changed
Parts:
- C4: value 10nF -> 100pF
Other:
- note added: "tune L4 for for better PLL margin"
Changed lines of the file:
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@@
 <part name="GND32" library="OSSI" deviceset="GND" device=""/>
 <part name="F1" library="OSSI" deviceset="LFCN-160" device=""/>
-<part name="C4" library="OSSI" deviceset="C" device="0603(1608)" value="10nF"/>
+<part name="C4" library="OSSI" deviceset="C" device="0603(1608)" value="100pF"/>
 <part name="GND33" library="OSSI" deviceset="GND" device=""/>
 <part name="GND34" library="OSSI" deviceset="GND" device=""/>
@@
 <sheet>
 <plain>
+<text x="193.04" y="96.52" size="1.778" layer="94">tune L4 for for better PLL margin</text>
 </plain>
 <instances>

Commit message: comms names renumbred
Other:
- note added: "Clock signal on Y is a bit distored"
Changed lines of the file:
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@@
 <plain>
 <text x="193.04" y="96.52" size="1.778" layer="94">tune L4 for for better PLL margin</text>
+<text x="86.36" y="106.68" size="1.778" layer="94">Clock signal on Y is a bit distored</text>
 </plain>
 <instances>
