File: OSSIComms/OSSICommsBeaconNewNew/OSSIBeaconNewNew.sch (EAGLE design)
At the start: 116 parts, among them Q1 NX-3215, U1 ADL5530, U10 MCP1700_SOT23, U2 MAX890L, U3 NC7SZ04, U4 ADF7012, U5 MAX6369, U6 MSP430F2132, U7 OPA2347, U8 TPS3838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

Commit message: all values for tuned results are updated
Parts:
- C33: value TBD -> 100nF
- C4: value 100pF -> 0R
- L4: value 10nH -> 8.2nH
Other:
- note added: "DC blocking cap is added on Front panel"
- note added: "External inductor is tuned to 8.2nH"
- note added: "with 8.2nH, PLL lock for all vco bias and adj are observed"
Changed lines of the file:
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@@
 <part name="R29" library="OSSI" deviceset="R" device="0603(1608)" value="DNP"/>
 <part name="R17" library="OSSI" deviceset="R" device="0603(1608)" value="100k"/>
-<part name="C33" library="OSSI" deviceset="C" device="0603(1608)" value="TBD"/>
+<part name="C33" library="OSSI" deviceset="C" device="0603(1608)" value="100nF"/>
 <part name="C30" library="OSSI" deviceset="C" device="0603(1608)" value="TBD"/>
 <part name="GND12" library="OSSI" deviceset="GND" device=""/>
@@
 <part name="C16" library="OSSI" deviceset="C" device="0603(1608)" value="1nF"/>
 <part name="VCCRF6" library="OSSI" deviceset="VCCRF" device=""/>
-<part name="L4" library="OSSI" deviceset="L" device="0603(1608)" value="10nH"/>
+<part name="L4" library="OSSI" deviceset="L" device="0603(1608)" value="8.2nH"/>
 <part name="C25" library="OSSI" deviceset="C" device="0603(1608)" value="22nF"/>
 <part name="R8" library="OSSI" deviceset="R" device="0603(1608)" value="3.6k"/>
@@
 <part name="GND32" library="OSSI" deviceset="GND" device=""/>
 <part name="F1" library="OSSI" deviceset="LFCN-160" device=""/>
-<part name="C4" library="OSSI" deviceset="C" device="0603(1608)" value="100pF"/>
+<part name="C4" library="OSSI" deviceset="C" device="0603(1608)" value="0R"/>
 <part name="GND33" library="OSSI" deviceset="GND" device=""/>
 <part name="GND34" library="OSSI" deviceset="GND" device=""/>
@@
 <text x="101.6" y="175.26" size="1.778" layer="94">PA Off by default</text>
 <text x="134.62" y="177.8" size="1.778" layer="94">Current limited to 220mA</text>
+<text x="213.36" y="116.84" size="1.778" layer="94">DC blocking cap is added on Front panel</text>
 </plain>
 <instances>
@@
 <text x="193.04" y="96.52" size="1.778" layer="94">tune L4 for for better PLL margin</text>
 <text x="86.36" y="106.68" size="1.778" layer="94">Clock signal on Y is a bit distored</text>
+<text x="193.04" y="93.98" size="1.778" layer="94">External inductor is tuned to 8.2nH </text>
+<text x="177.8" y="91.44" size="1.778" layer="94">with 8.2nH, PLL lock for all vco bias and adj are observed</text>
 </plain>
 <instances>

Commit message: design files are added
Parts:
- C1: value (none) -> DNP
- R1: value 511 -> DNP
Other:
- note added: "TCXO signal is needed to be boosted via NC7SZ04 to feed OSC input of ADF7012"
Changed lines of the file:
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@@
 <?xml version="1.0" encoding="utf-8"?>
 <!DOCTYPE eagle SYSTEM "eagle.dtd">
-<eagle version="6.1">
+<eagle version="6.5.0">
 <drawing>
 <settings>
@@
 <part name="X6" library="OSSI" deviceset="M03" device="PTH"/>
 <part name="GND35" library="OSSI" deviceset="GND" device=""/>
-<part name="R1" library="OSSI" deviceset="R" device="WSL1206" value="511"/>
-<part name="C1" library="OSSI" deviceset="C" device="0805(2012)"/>
+<part name="R1" library="OSSI" deviceset="R" device="WSL1206" value="DNP"/>
+<part name="C1" library="OSSI" deviceset="C" device="0805(2012)" value="DNP"/>
 <part name="GND37" library="OSSI" deviceset="GND" device=""/>
 <part name="TP1" library="OSSI" deviceset="TP" device=""/>
@@
 <text x="193.04" y="93.98" size="1.778" layer="94">External inductor is tuned to 8.2nH </text>
 <text x="177.8" y="91.44" size="1.778" layer="94">with 8.2nH, PLL lock for all vco bias and adj are observed</text>
+<text x="38.1" y="86.36" size="1.778" layer="94">TCXO signal is needed to be boosted via NC7SZ04 to feed OSC input of ADF7012</text>
 </plain>
 <instances>
