File: OSSIComms/OSSICommsBeaconNewNew/OSSIBeaconNewNew.brd (EAGLE design)
At the start: 92 x 92 mm, 116 parts, among them Q1 NX-3215, U1 ADL5530, U10 MCP1700_SOT23, U2 MAX890L, U3 NC7SZ04, U4 ADF7012, U5 MAX6369, U6 MSP430F2132, U7 OPA2347, U8 TPS3838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

Commit message: all values for tuned results are updated
Parts:
- C33: value TBD -> 100nF
- C4: value 100pF -> 0R
- L4: value 10nH -> 8.2nH
Changed lines of the file:
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@@
 <attribute name="VALUE" x="23.749" y="48.387" size="1.27" layer="27" rot="R180"/>
 </element>
-<element name="C33" library="OSSI" package="C0603(1608)" value="TBD" x="22.86" y="37.465" smashed="yes" rot="R180">
+<element name="C33" library="OSSI" package="C0603(1608)" value="100nF" x="22.86" y="37.465" smashed="yes" rot="R180">
 <attribute name="NAME" x="21.209" y="37.846" size="1.27" layer="25" font="vector" rot="R180"/>
 <attribute name="VALUE" x="23.749" y="39.497" size="1.27" layer="27" rot="R180"/>
@@
 <attribute name="VALUE" x="63.754" y="22.352" size="1.27" layer="27" rot="R180"/>
 </element>
-<element name="L4" library="OSSI" package="L0603(1608)" value="10nH" x="45.085" y="22.86" smashed="yes" rot="R90">
+<element name="L4" library="OSSI" package="L0603(1608)" value="8.2nH" x="45.085" y="22.86" smashed="yes" rot="R90">
 <attribute name="NAME" x="44.196" y="21.971" size="1.27" layer="25" font="vector" rot="R90"/>
 <attribute name="VALUE" x="47.117" y="21.971" size="1.27" layer="27" rot="R90"/>
@@
 <attribute name="VALUE" x="24.050003125" y="25.050003125" size="1.778" layer="27" rot="R180"/>
 </element>
-<element name="C4" library="OSSI" package="C0603(1608)" value="100pF" x="15.24" y="19.05" smashed="yes" rot="R180">
+<element name="C4" library="OSSI" package="C0603(1608)" value="0R" x="15.24" y="19.05" smashed="yes" rot="R180">
 <attribute name="NAME" x="16.764" y="17.526" size="1.27" layer="25" font="vector" rot="R180"/>
 <attribute name="VALUE" x="16.129" y="21.082" size="1.27" layer="27" rot="R180"/>

Commit message: design files are added
Parts:
- C1: value (none) -> DNP
- R1: value 511 -> DNP
Changed lines of the file:
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@@
 <?xml version="1.0" encoding="utf-8"?>
 <!DOCTYPE eagle SYSTEM "eagle.dtd">
-<eagle version="6.1">
+<eagle version="6.5.0">
 <drawing>
 <settings>
@@
 </class>
 </classes>
-<designrules>
+<designrules name="default">
 <description language="de">&lt;b&gt;EAGLE Design Rules&lt;/b&gt;
 &lt;p&gt;
@@
 <attribute name="VALUE" x="92.075" y="27.305" size="1.27" layer="27" rot="R90"/>
 </element>
-<element name="R1" library="OSSI" package="WSL1206" value="511" x="8.89" y="78.105" smashed="yes" rot="R90">
+<element name="R1" library="OSSI" package="WSL1206" value="DNP" x="8.89" y="78.105" smashed="yes" rot="R90">
 <attribute name="NAME" x="9.525" y="74.295" size="1.27" layer="25" font="vector" rot="R90"/>
 <attribute name="VALUE" x="11.43" y="74.295" size="1.27" layer="27" rot="R90"/>
 </element>
-<element name="C1" library="OSSI" package="C0805(2012)" value="" x="6.35" y="78.105" smashed="yes" rot="R270">
+<element name="C1" library="OSSI" package="C0805(2012)" value="DNP" x="6.35" y="78.105" smashed="yes" rot="R270">
 <attribute name="NAME" x="5.461" y="76.454" size="1.27" layer="25" font="vector" rot="R270"/>
 <attribute name="VALUE" x="4.064" y="78.994" size="1.27" layer="27" rot="R270"/>
