File: OSSIComms/OSSICommsNew/OSSICommsNew.brd (EAGLE design)
At the start: 94 x 94 mm, 188 parts, among them Q2 NX-3215, U1 MAX890L, U10 LMZ10503EXT, U11 OPA347, U14 RF5110G, U16 MAX2640, U2 ADF7021-N, U3 ADF7021-N, U4 PE4259, U5 MSP430F1611, U6 MAX6369, U7 TPS3838, U8 MCP1700_SOT23, U9 MAX869L, X1 ESQ-126-38-G-D, X2 JTAG10PINMINI-H, X3 P-PAD-S, X4 P-PAD-S, X5 RFCON-MCX-R/A, X7 5268-03

Commit message: schematics renumbered
Parts:
- removed C94: 330pF, OSSI:C0603(1608)
- removed C95: 1nF, OSSI:C0603(1608)
- removed C96: 10nF, OSSI:C0603(1608)
- removed R75: 0, OSSI:R0603(1608)
- removed U14: RF5110G, OSSI:RF5110G
- removed U16: MAX2640, OSSI:SOT23-6
- added C73, C77: 100nF, OSSI:C0603(1608)
- added C76: 10nF, OSSI:C0603(1608)
- added R44: 100k, OSSI:R0603(1608)
- added U12: MAX890L, OSSI:SO8
- added U13: MCP1700_SOT23, OSSI:SOT23
- C1: value 1uF -> 6.8pF
- C10: value 100nF -> (none)
- C11: value 470pF 0805 -> 3.3uF; device OSSI:C0805(2012) -> OSSI:C1210-TMK325
- C12: value 10uF -> 10pF; device OSSI:C1206-GCM31 -> OSSI:C0603(1608)
- C13: value 12.5pF -> 1nF
- C14: value 12.5pF -> 15pF
- C15: value 10nF -> (none)
- C16: value 100nF -> DNP
- C17: value 10nF -> DNP
- C18, C25: value 100nF -> 8.2pF
- C19: value 10nF -> 12pF
- C2: value 13pF -> DNP
- C20: value 22nF -> 8.2pF
- C21: value 100nF -> 22pF
- C22: value 100nF -> 2pF
- C23: value 100pF -> DNP
- C24, C3: value 100nF -> 13pF
- C26: value 10nF -> 56pF
- C27: value 100nF -> 330pF
- C29, C70: value 100nF -> 100pF
- C30: value 10nF -> 47pF
- C31: value 22nF -> 1nF
- C32, C35, C36, C67: value 100nF -> 10nF
- C33: value 100nF -> 1nF
- C34: value 100pF -> 100nF
- C37: value 100nF -> 3.3uF; device OSSI:C0603(1608) -> OSSI:C1210-TMK325
- C38: value 100pF -> 180pF
- C39, C93: value 15pF -> 100nF
- C4: value 10uF, LDO Tantal 16V -> 15pF; device OSSI:C1206(3216)-A -> OSSI:C0603(1608)
- C40: value 8.2pF -> 100nF
- C41: value 12pF -> (none); device OSSI:C0603(1608) -> OSSI:C1210-GCM32
- C42: value 8.2pF -> 22uF,1210; device OSSI:C0603(1608) -> OSSI:C1210-GCM32
- C43: value 1.2nF -> 10nF
- C44: value 100nF -> 100uF,1210; device OSSI:C0603(1608) -> OSSI:C0805(2012)
- C45: value 10nF -> (none); device OSSI:C0603(1608) -> OSSI:C1210-GCM32
- C46: value 1.2nF -> (none); device OSSI:C0603(1608) -> OSSI:C1210-GCM32
- C48, C54, C88: value 10nF -> 100nF
- C49: value 6.8pF -> 100nF
- C5: value 10uF, LDO Tantal 16V -> DNP; device OSSI:C1206(3216)-A -> OSSI:C0603(1608)
- C50, C66: value DNP -> 100nF
- C51, C56: value DNP -> 10nF
- C52, C69: value (none) -> 100nF
- C53: value (none) -> 100pF
- C55, C71: value 100nF -> 22nF
- C57: value DNP -> 1.2nF
- C58: value 22uF,1210 -> 100nF; device OSSI:C1210-GCM32 -> OSSI:C0603(1608)
- C59: value (none) -> 10nF; device OSSI:C1210-GCM32 -> OSSI:C0603(1608)
- C6: value 13pF -> 10uF; device OSSI:C0603(1608) -> OSSI:C1206-GCM31
- C60: value (none) -> 100nF; device OSSI:C1210-GCM32 -> OSSI:C0603(1608)
- C61: value (none) -> 22pF; device OSSI:C1210-GCM32 -> OSSI:C0603(1608)
- C62: value 100uF,1210 -> 10nF; device OSSI:C0805(2012) -> OSSI:C0603(1608)
- C64: value 180pF -> 100nF
- C7: value 100nF -> 470pF 0805; device OSSI:C0603(1608) -> OSSI:C0805(2012)
- C72: value 22uF,1210 -> 1.2nF; device OSSI:C1210-GCM32 -> OSSI:C0603(1608)
- C79: value 22pF -> 10nF
- C8: value 100nF -> 1500pF
- C80: value 8.2pF -> 12.5pF
- C81: value 47pF -> 12.5pF
- C82: value 1nF -> 100nF
- C83: value 3.3uF -> 100nF; device OSSI:C1210-TMK325 -> OSSI:C0603(1608)
- C84: value 22pF -> 100nF
- C85: value 2pF -> 100nF
- C86: value 56pF -> 100nF
- C87: value 10nF -> 1uF
- C89: value 10nF -> 10uF, LDO Tantal 16V; device OSSI:C0603(1608) -> OSSI:C1206(3216)-A
- C9: value 1500pF -> (none)
- C90: value 3.3uF -> 10uF, LDO Tantal 16V; device OSSI:C1210-TMK325 -> OSSI:C1206(3216)-A
- C91: value 1nF -> 10nF
- C92: value 10pF -> 22uF,1210; device OSSI:C0603(1608) -> OSSI:C1210-GCM32
- L1: value 26nH -> 27nH
- L11: value 3.9nH -> 11nH
- L12: value 1.5nH -> 11nH
- L13: value 0 Ohm -> 3.9nH; device OSSI:L0805(2012) -> OSSI:L0603(1608)
- L14: value (none) -> 26nH
- L15: value (none) -> 39nH 3012, 1A rating; device OSSI:L0603(1608) -> OSSI:NR3012
- L16: value 330uH -> 0 Ohm; device OSSI:LQH32CN331K23L -> OSSI:L0805(2012)
- L2, L3: value 11nH -> (none)
- L4: value 27nH -> (none)
- L5: value 39nH 3012, 1A rating -> 47nH; device OSSI:NR3012 -> OSSI:L0603(1608)
- L6: value 47nH -> (none)
- L7: value (none) -> 330uH; device OSSI:L0603(1608) -> OSSI:LQH32CN331K23L
- L9: value (none) -> 1.5nH
- R1: value TBD -> 100k
- R10: value 3.6k -> 1.5k
- R11: value 3.9 -> TBD
- R12: value 1.1k -> 100k
- R13: value 3.6k -> 100k
- R14: value 3.9 -> 1.5k
- R15: value 280 -> 100k
- R16: value 100 -> 22k
- R17: value 280 -> 3.9
- R18: value 100 -> 3.6k
- R19: value 1.5k -> 1.1k
- R2, R3: value 100k -> 1.5k
- R20: value 100k -> 280
- R21: value 15.968k -> 100
- R22: value 49.9k -> 3.6k
- R23: value 4.12k -> 3.9
- R24: value TBD -> 1.1k
- R25: value 1.5k -> 280
- R26: value 250 -> 100
- R28: value 100k -> 4.7k
- R29: value 1k -> 4.7k
- R30: value 10k -> 250
- R32: value 100k -> 10k
- R33: value 1.5k -> 4.7k
- R34: value 180 -> 4.7k
- R35: value 470k -> 4.7k
- R36: value 11nH -> 470k
- R37: value 22k -> 1.5k
- R38: value 100k -> 1k
- R4: value 470k -> 180
- R41: value 4.7k -> 0
- R42: value 4.7k -> TBD
- R43: value 4.7k -> 100k
- R5: value 4.7k -> 11nH
- R6: value 1.5k -> 4.12k
- R7: value 1.5k -> 470k
- R8: value 4.7k -> 15.968k
- R9: value 1.1k -> 49.9k
- U1: value MAX890L -> MAX2640; device OSSI:SO8 -> OSSI:SOT23-6
- U10: value LMZ10503EXT -> MAX6369; device OSSI:TO-PMOD-7 -> OSSI:SOT23-8
- U11: value OPA347 -> TPS3838
- U2: value ADF7021-N -> PE4259; device OSSI:LFCSP48 -> OSSI:SC70-6
- U3: value ADF7021-N -> RF5110G; device OSSI:LFCSP48 -> OSSI:RF5110G
- U4: value PE4259 -> OPA347; device OSSI:SC70-6 -> OSSI:SOT23-5DBV
- U5: value MSP430F1611 -> MAX869L; device OSSI:PM/PAG64 -> OSSI:16QSOP
- U6: value MAX6369 -> LMZ10503EXT; device OSSI:SOT23-8 -> OSSI:TO-PMOD-7
- U7: value TPS3838 -> ADF7021-N; device OSSI:SOT23-5DBV -> OSSI:LFCSP48
- U8: value MCP1700_SOT23 -> ADF7021-N; device OSSI:SOT23 -> OSSI:LFCSP48
- U9: value MAX869L -> MSP430F1611; device OSSI:16QSOP -> OSSI:PM/PAG64
- X2: value JTAG10PINMINI-H -> RFCON-MCX-R/A; device OSSI:M50-3200545 -> OSSI:MCX-R/A
- X3: value P-PAD-S -> (none); device OSSI:P-PAD-S -> OSSI:1X03
- X5: value RFCON-MCX-R/A -> 5268-03; device OSSI:MCX-R/A -> OSSI:5268-03
- X6: value (none) -> P-PAD-S; device OSSI:1X03 -> OSSI:P-PAD-S
- X7: value 5268-03 -> JTAG10PINMINI-H; device OSSI:5268-03 -> OSSI:M50-3200545
- moved H1 107.5 mm to (85.0, 85.0)
- moved H2 107.5 mm to (85.0, 9.00)
- moved H3 107.5 mm to (9.00, 85.0)
- moved H4 107.5 mm to (9.00, 9.00)
- moved X5 86.3 mm to (66.0, 83.8), turned to 0 degrees
- moved C5 85.3 mm to (15.2, 26.4), turned to 180 degrees
- moved C83 83.7 mm to (55.2, 86.4), turned to 90 degrees
- moved C59 79.4 mm to (13.0, 73.0), turned to 180 degrees
- moved C89 79.0 mm to (76.5, 81.3), turned to 0 degrees
- moved C88 77.5 mm to (76.2, 78.9), turned to 0 degrees
- moved C82 72.7 mm to (36.5, 80.6), turned to 90 degrees
- moved X2 72.7 mm to (7.94, 20.0), turned to 90 degrees
- moved C45 71.6 mm to (70.3, 21.3), turned to 0 degrees
- moved C60 71.4 mm to (11.4, 61.6), turned to 180 degrees
- moved C86 71.1 mm to (39.4, 85.1), turned to 90 degrees
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- renumbered Q2 to Q1, TCXO3 to TCXO1
Connections:
- net /RST: now also R40.2, R44.1, U11.4, U9.58; no longer R2.1, R8.2, U5.58, U7.4
- net 3.3VCOMMS: now also C84.1, C85.1, C86.1, C90.1, C91.1, C92.P$1, L16.1, R12.1, R32.2, R36.2, R44.2, U10.4, U10.5, U10.6, U10.8, U11.5, U13.2, U9.1, U9.64, X7.4; no longer C5.1, C54.1, C7.1, C70.1, C72.P$1, C8.1, L13.1, R2.2, R28.1, R30.2, R4.2, U5.1, U5.64, U6.4, U6.5, U6.6, U6.8, U7.5, U8.2, X2.4
- net COMMSRX_CE: now also U7.24, U9.21; no longer U3.24, U5.21
- net COMMSRX_CLK: now also R35.2, U7.35; no longer R42.2, U3.35
- net COMMSRX_CLKOUT: now also U7.36; no longer U3.36
- net COMMSRX_CPOUT: now also C62.1, R20.2, R21.2, U7.42; no longer C45.1, R15.2, R16.2, U3.42
- net COMMSRX_DATA: now also R34.2, U7.34; no longer R43.2, U3.34
- net COMMSRX_MUXOUT: now also U7.37, U9.13; no longer U3.37, U5.13
- net COMMSRX_RFIN: now also C3.1, L1.2, U7.6; no longer C2.1, L4.2, U3.6
- net COMMSRX_RFINB: now also C1.1, L1.1, U7.7; no longer C49.1, L4.1, U3.7
- net COMMSRX_SCLK: now also U7.28, U9.17; no longer U3.28, U5.17
- net COMMSRX_SDATA: now also U7.26, U9.19; no longer U3.26, U5.19
- net COMMSRX_SLE: now also U7.25, U9.20; no longer U3.25, U5.20
- net COMMSRX_SREAD: now also U7.27, U9.18; no longer U3.27, U5.18
- net COMMSRX_SWD: now also U7.33, U9.16; no longer U3.33, U5.16
- net COMMSRX_TCXO: now also C61.2, U7.39; no longer C79.2, U3.39
- net COMMSRX_VCOIN: now also C57.1, R20.1, U7.1; no longer C43.1, R15.1, U3.1
- net COMMSTX_CE: now also U8.24, U9.37; no longer U2.24, U5.37
- net COMMSTX_CLK: now also R28.2, U8.35; no longer R41.2, U2.35
- net COMMSTX_CLKOUT: now also U8.36; no longer U2.36
- net COMMSTX_CPOUT: now also C75.1, R25.2, R26.2, U8.42; no longer C48.1, R17.2, R18.2, U2.42
- net COMMSTX_DATA: now also R29.2, U8.34; no longer R40.2, U2.34
- net COMMSTX_MUXOUT: now also U8.37, U9.22; no longer U2.37, U5.22
- net COMMSTX_RFOUT: now also C24.1, L14.1, U8.4; no longer C6.1, L1.1, U2.4
- net COMMSTX_SCLK: now also U8.28, U9.25; no longer U2.28, U5.25
- net COMMSTX_SDATA: now also U8.26, U9.27; no longer U2.26, U5.27
- net COMMSTX_SLE: now also U8.25, U9.36; no longer U2.25, U5.36
- net COMMSTX_SREAD: now also U8.27, U9.26; no longer U2.27, U5.26
- net COMMSTX_TCXO: now also U8.39; no longer U2.39
- net COMMSTX_VCOIN: now also C72.1, R25.1, U8.1; no longer C46.1, R17.1, U2.1
- net COMMS_-FAULT: now also U12.8; no longer U1.8
- net COMMS_-RST: now also C83.1, U10.7, U11.3; no longer C71.1, U6.7, U7.3
- net COMMS_OFF: now also C87.1, R43.2, U12.3; no longer C1.1, R3.2, U1.3
- net COMMS_SCL: now also R32.1, X3.2; no longer R26.1, X6.2
- net COMMS_SDA: now also X3.1; no longer X6.1
- net GND: now also C11.P$2, C12.2, C16.1, C17.1, C2.2, C20.2, C21.2, C23.1, C28.1, C31.2, C32.1, C36.1, C37.P$2, C39.2, C41.P$2, C42.P$2, C45.P$2, C46.P$2, C5.2, C51.2, C52.2, C53.2, C56.2, C57.2, C58.2, C59.2, C6.P$2, C60.2, C64.2, C69.2, C72.2, C73.2, C76.2, C77.2, C79.2, C80.2, C83.2, C86.2, C87.2, C88.2, C89.2, C92.P$2, L2.2, L4.2, R13.2, R17.1, R18.2, R19.2, R22.1, R23.1, R4.1, R41.2, R42.1, R43.1, R7.2, R8.2, U1.2, U1.3, U1.5, U10.2, U11.1, U12.4, U13.1, U2.2, U3.2, U3.4, U3.TPAD, U5.8, U6.4, U6.PAD, U7.12, U7.19, U7.22, U7.29, U7.45, U7.47, U7.5, U7.EXP, U8.12, U8.19, U8.22, U8.29, U8.45, U8.47, U8.5, U8.6, U8.7, U8.EXP, U9.53, U9.62, U9.63, X2.2, X2.3, X2.4, X2.5, X3.3, X5.1, X7.9; no longer C10.2, C11.2, C12.P$2, C15.2, C16.2, C17.2, C23.2, C24.2, C25.2, C26.2, C28.2, C3.2, C36.2, C37.2, C38.2, C4.2, C41.2, C42.2, C45.2, C46.2, C51.1, C54.2, C55.2, C56.1, C57.1, C58.P$2, C59.P$2, C60.P$2, C61.P$2, C68.2, C71.2, C72.P$2, C8.2, C83.P$2, C87.1, C88.1, C89.1, C90.P$2, C92.2, C94.2, C95.2, C96.2, L10.2, L15.2, R10.2, R12.1, R13.1, R14.1, R21.2, R3.1, R32.1, R34.1, R35.2, R38.2, R75.2, R9.2, U1.4, U10.4, U10.PAD, U14.2, U14.4, U14.TPAD, U16.2, U16.3, U16.5, U2.12, U2.19, U2.22, U2.29, U2.45, U2.47, U2.5, U2.6, U2.7, U2.EXP, U3.12, U3.19, U3.22, U3.29, U3.45, U3.47, U3.5, U3.EXP, U5.53, U5.62, U5.63, U6.2, U7.1, U7.2, U8.1, U9.8, X2.9, X5.2, X5.3, X5.4, X5.5, X6.3, X7.1
- net LED1: now also U9.50; no longer U5.50
- net N$1: now also C60.1, U7.41; no longer C16.1, U3.41
- net N$10: now also C49.1, U7.11; no longer C25.1, U3.11
- net N$11: now also C88.1, C89.1, U12.6, U12.7, U13.3; no longer C3.1, C4.1, U1.6, U1.7, U8.3
- net N$12: now also R42.2, U12.5; no longer R1.2, U1.5
- net N$13: now also C82.1, U9.7; no longer C10.1, U5.7
- net N$14: now also C4.2, U1.4; no longer C39.2, U16.4
- net N$15: now also C5.1, L6.1; no longer C50.1, L9.1
- net N$16: now also C8.2; no longer C9.2
- net N$17: now also U9.57, X7.7; no longer U5.57, X2.7
- net N$18: now also U9.56, X7.5; no longer U5.56, X2.5
- net N$19: now also U9.55, X7.3; no longer U5.55, X2.3
- net N$2: now also R40.1, X7.10; no longer R8.1, X2.10
- net N$20: now also U9.54, X7.1; no longer U5.54, X2.1
- net N$21: now also C9.1, L4.1, L6.2; no longer C53.1, L10.1, L9.2
- net N$22: now also C55.1, U7.48; no longer C20.1, U3.48
- net N$23: now also C17.2, L10.2; no longer C51.2, L7.2
- net N$24: now also R19.1, U7.8; no longer R9.1, U3.8
- net N$25: now also R18.1, U7.10; no longer R10.1, U3.10
- net N$26: now also C54.2, R17.2; no longer C21.2, R11.2
- net N$27: now also C71.1, U8.48; no longer C31.1, U2.48
- net N$28: now also R22.2, U8.10; no longer R13.2, U2.10
- net N$29: now also C68.2, R23.2; no longer C32.2, R14.2
- net N$3: now also C65.1, U8.11; no longer C36.1, U2.11
- net N$30: now also R24.2, U8.8; no longer R12.2, U2.8
- net N$31: now also C77.1, U8.41; no longer C27.1, U2.41
- net N$32: now also C66.1, U8.31; no longer C29.1, U2.31
- net N$33: now also C20.1, C25.1, L12.2, R4.2; no longer C42.1, C80.1, L3.2, R34.2
- net N$34: now also C68.1, C71.2, U8.2; no longer C31.2, C32.1, U2.2
- net N$35: now also C54.1, C55.2, U7.2; no longer C20.2, C21.1, U3.2
- net N$36: now also C18.1, C24.2, L11.1; no longer C40.1, C6.2, L2.1
- net N$37: now also C19.1, L11.2, L12.1; no longer C41.1, L2.2, L3.1
- net N$38: now also C73.1, R26.1; no longer C47.1, R18.1
- net N$39: now also C15.2, C16.2; no longer C52.2, C57.2
- net N$4: now also C23.2, C26.2, L10.1; no longer C56.2, C86.2, L7.1
- net N$40: now also C58.1, R21.1; no longer C44.1, R16.1
- net N$41: now also C10.2, U2.5; no longer C69.2, U4.5
- net N$42: now also R2.2, U2.4; no longer R6.2, U4.4
- net N$43: now also C4.1, L2.1, L3.2; no longer C39.1, L14.2, L15.1
- net N$44: now also R3.1, U2.6; no longer R19.1, U4.6
- net N$45: now also LED1.A, R38.2; no longer LED2.A, R29.2
- net N$46: now also C10.1, X2.1; no longer C69.1, X5.1
- net N$47: now also C40.1, R15.1, U5.7; no longer C65.1, R20.1, U9.7
- net N$48: now also R38.1, U9.49; no longer R29.1, U5.49
- net N$49: now also LED2.A; no longer LED1.A
- net N$5: now also C81.1, U9.8; no longer C13.1, U5.8
- net N$50: now also C43.1, U6.3; no longer C63.1, U10.3
- net N$51: now also R10.1; no longer R25.1
- net N$52: now also C41.P$1, C42.P$1, U5.11, U5.14, U5.15, U5.2, U5.3, U5.6, U6.1, U6.2; no longer C58.P$1, C61.P$1, U10.1, U10.2, U9.11, U9.14, U9.15, U9.2, U9.3, U9.6
- net N$53: now also R6.2, R8.1, R9.2, U6.5; no longer R21.1, R22.2, R23.2, U10.5
- net N$54: now also C38.2, R6.1; no longer C64.2, R23.1
- net N$55: now also R11.2, U5.9; no longer R24.2, U9.9
- net N$56: now also U9.35, X5.3; no longer U5.35, X7.3
- net N$57: now also U9.34, X5.2; no longer U5.34, X7.2
- net N$58: now also C15.1, U2.1; no longer C52.1, U4.1
- net N$59: now also C9.2, U2.3; no longer C53.2, U4.3
- net N$6: now also C80.1, U9.9; no longer C14.1, U5.9
- net N$60: now also U9.29; no longer U5.29
- net N$61: now also R30.2, U9.31; no longer R26.2, U5.31
- net N$62: now also C2.1, C3.2, L3.1; no longer C2.2, C66.1, L14.1
- net N$63: now also R34.1, U9.15; no longer R43.1, U5.15
- net N$64: now also R35.1, U9.14; no longer R42.1, U5.14
- net N$65: now also R28.1, U9.23; no longer R41.1, U5.23
- net N$66: now also C61.1; no longer C79.1
- net N$67: now also R29.1, U9.24; no longer R40.1, U5.24
- net N$69: now also U10.1, U9.42; no longer U5.42, U6.1
- net N$7: now also L5.1, U1.1; no longer L6.1, U16.1
- net N$70: now also C39.1, R14.2, U4.3; no longer C67.1, R33.2, U11.3
- net N$71: now also C21.1, C22.1, C26.1, L13.2; no longer C84.1, C85.1, C86.1, L11.2
- net N$72: now also L9.2, U3.5, U3.6; no longer L12.2, U14.5, U14.6
- net N$73: now also C25.2, U3.3; no longer C80.2, U14.3
- net N$74: now also C90.2, R41.1; no longer C5.2, R75.1
- net N$75: now also L13.1, L15.P$1, U3.10, U3.11, U3.12, U3.9; no longer L11.1, L5.P$1, U14.10, U14.11, U14.12, U14.9
- net N$76: now also U4.1; no longer U11.1
- net N$77: now also U9.33, X6.1; no longer U5.33, X3.1
- net N$78: now also U9.32; no longer U5.32
- net N$79: now also C14.1, L7.P$2, L9.1; no longer C93.1, L12.1, L16.P$2
- net N$8: now also C8.1, L5.2; no longer C9.1, L6.2
- net N$80: now also R5.1, U3.1; no longer R36.1, U14.1
- net N$9: now also C50.1, U7.31; no longer C18.1, U3.31
- net OBC_-FAULT: now also R33.2, R36.1; no longer R4.1, R5.2
- net OBC_-FAULT_IN: now also R33.1, U9.12; no longer R5.1, U5.12
- net OBC_OFF: now also R37.2; no longer R7.2
- net OBC_OFF_OUT: now also R37.1, U9.2; no longer R7.1, U5.2
- net PA_-FAULT: now also R12.2, U5.10; no longer R28.2, U9.10
- net PA_BIAS: now also R13.1, R14.1, R16.2, U9.5; no longer R33.1, R37.2, R38.1, U5.5
- net PA_ON: now also R10.2, R7.1, U9.40; no longer R25.2, R35.1, U5.40
- net RX_ON: now also U9.39; no longer U5.39
- net STRUT_GND: now also H4.B3,2; no longer H1.B3,2
- net TX_ON: now also R1.2, R2.1, U9.38; no longer R32.2, R6.1, U5.38
- net VAPC: now also C28.2, C32.2, U3.15, U3.16; no longer C88.2, C89.2, U14.15, U14.16
- net VBUS: now also R15.2, U12.1, U12.2, U5.1, U5.12, U5.13, U5.16, U5.4, U5.5; no longer R20.2, U1.1, U1.2, U9.1, U9.12, U9.13, U9.16, U9.4, U9.5
- net VCCRF: now also C29.1, C48.1, C51.1, C52.1, C53.1, C56.1, C59.1, C6.P$1, C63.1, C64.1, C67.1, C69.1, C7.1, C70.1, C76.1, C79.1, C93.1, L14.2, L16.2, R3.2, U1.6, U7.3, U7.32, U7.40, U7.43, U7.9, U8.3, U8.32, U8.40, U8.43, U8.9; no longer C11.1, C12.P$1, C15.1, C17.1, C19.1, C22.1, C23.1, C24.1, C26.1, C28.1, C30.1, C33.1, C35.1, C37.1, C38.1, C55.1, C75.1, L1.2, L13.2, R19.2, U16.6, U2.3, U2.32, U2.40, U2.43, U2.9, U3.3, U3.32, U3.40, U3.43, U3.9
- net VCOMMS_PA: now also C11.P$1, C12.1, C13.1, C27.1, C30.1, C31.1, C33.1, C35.1, C36.2, C37.P$1, C38.1, C44.1, C45.P$1, C46.P$1, C47.1, L15.P$2, L7.P$1, R16.1, R5.2, R9.1, U3.14, U4.5, U6.6, U6.7; no longer C59.P$1, C60.P$1, C62.1, C64.1, C68.1, C81.1, C82.1, C83.P$1, C87.2, C90.P$1, C91.1, C92.1, C94.1, C95.1, C96.1, L16.P$1, L5.P$2, R22.1, R36.2, R37.1, U10.6, U10.7, U11.5, U14.14

Commit message: LNA gain measured to 15.5dB and R / L values are fixed
Parts:
- C4: value 15pF -> 8.2pF
- C8: value 1500pF -> 1000pF
- L5: value 47nH -> 39nH
Changed lines of the file:
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@@
 <attribute name="VALUE" x="46.89475" y="82.51825" size="1.27" layer="28" rot="MR180"/>
 </element>
-<element name="C8" library="OSSI" package="C0603(1608)" value="1500pF" x="17.78" y="33.3375" smashed="yes" rot="R270">
+<element name="C8" library="OSSI" package="C0603(1608)" value="1000pF" x="17.78" y="33.3375" smashed="yes" rot="R270">
 <attribute name="NAME" x="14.0335" y="32.639" size="1.27" layer="25" font="vector"/>
 <attribute name="VALUE" x="15.748" y="34.2265" size="1.27" layer="27" rot="R270"/>
 </element>
-<element name="L5" library="OSSI" package="L0603(1608)" value="47nH" x="17.78" y="36.195" smashed="yes" rot="R270">
+<element name="L5" library="OSSI" package="L0603(1608)" value="39nH" x="17.78" y="36.195" smashed="yes" rot="R270">
 <attribute name="NAME" x="14.351" y="35.814" size="1.27" layer="25" font="vector"/>
 <attribute name="VALUE" x="15.748" y="37.084" size="1.27" layer="27" rot="R270"/>
@@
 <attribute name="VALUE" x="15.24" y="39.6875" size="1.27" layer="27" rot="R90"/>
 </element>
-<element name="C4" library="OSSI" package="C0603(1608)" value="15pF" x="19.685" y="44.1325" smashed="yes" rot="R270">
+<element name="C4" library="OSSI" package="C0603(1608)" value="8.2pF" x="19.685" y="44.1325" smashed="yes" rot="R270">
 <attribute name="NAME" x="20.701" y="43.434" size="1.27" layer="25" font="vector"/>
 <attribute name="VALUE" x="17.653" y="45.0215" size="1.27" layer="27" rot="R270"/>

Commit message: COMMS PA setting fixed!
Parts:
- C21: value 22pF -> 10pF
- C22: value 2pF -> 6pF
- C25: value 8.2pF -> 56pF
- L10, L8: value (none) -> 0R
- L7: value 330uH -> 0R
Changed lines of the file:
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@@
 <layer number="21" name="tPlace" color="7" fill="1" visible="yes" active="yes"/>
 <layer number="22" name="bPlace" color="7" fill="1" visible="yes" active="yes"/>
-<layer number="23" name="tOrigins" color="15" fill="1" visible="no" active="yes"/>
+<layer number="23" name="tOrigins" color="15" fill="1" visible="yes" active="yes"/>
 <layer number="24" name="bOrigins" color="15" fill="1" visible="no" active="yes"/>
 <layer number="25" name="tNames" color="12" fill="1" visible="no" active="yes"/>
@@
 <attribute name="VALUE" x="47.690021875" y="17.9705" size="1.27" layer="27"/>
 </element>
-<element name="C25" library="OSSI" package="C0603(1608)" value="8.2pF" x="47.14875" y="14.76375" smashed="yes" rot="R180">
+<element name="C25" library="OSSI" package="C0603(1608)" value="56pF" x="47.14875" y="14.76375" smashed="yes" rot="R180">
 <attribute name="NAME" x="52.16525" y="15.46225" size="1.27" layer="25" font="vector" rot="R180"/>
 <attribute name="VALUE" x="48.03775" y="16.79575" size="1.27" layer="27" rot="R180"/>
@@
 </element>
 <element name="C37" library="OSSI" package="C1210-TMK325" value="3.3uF" x="33.9725" y="5.3975" smashed="yes" rot="R180"/>
-<element name="C21" library="OSSI" package="C0603(1608)" value="22pF" x="32.54375" y="12.065" smashed="yes" rot="R270">
+<element name="C21" library="OSSI" package="C0603(1608)" value="10pF" x="32.54375" y="12.065" smashed="yes" rot="R270">
 <attribute name="NAME" x="31.84525" y="10.7315" size="1.27" layer="25" font="vector" rot="R270"/>
 <attribute name="VALUE" x="30.51175" y="12.954" size="1.27" layer="27" rot="R270"/>
 </element>
-<element name="C22" library="OSSI" package="C0603(1608)" value="2pF" x="30.63875" y="12.065" smashed="yes" rot="R270">
+<element name="C22" library="OSSI" package="C0603(1608)" value="6pF" x="30.63875" y="12.065" smashed="yes" rot="R270">
 <attribute name="NAME" x="30.25775" y="10.7315" size="1.27" layer="25" font="vector" rot="R270"/>
 <attribute name="VALUE" x="28.60675" y="12.954" size="1.27" layer="27" rot="R270"/>
@@
 <attribute name="VALUE" x="23.780003125" y="24.209996875" size="1.778" layer="27" rot="R90"/>
 </element>
-<element name="L10" library="OSSI" package="L0603(1608)" value="" x="27.305" y="14.605" smashed="yes" rot="R180">
+<element name="L10" library="OSSI" package="L0603(1608)" value="0R" x="27.305" y="14.605" smashed="yes" rot="R180">
 <attribute name="NAME" x="28.5115" y="17.2085" size="1.27" layer="25" font="vector" rot="R180"/>
 <attribute name="VALUE" x="28.194" y="16.637" size="1.27" layer="27" rot="R180"/>
 </element>
-<element name="L8" library="OSSI" package="L0603(1608)" value="" x="24.4475" y="14.605" smashed="yes" rot="R180">
+<element name="L8" library="OSSI" package="L0603(1608)" value="0R" x="24.4475" y="14.605" smashed="yes" rot="R180">
 <attribute name="NAME" x="25.654" y="17.2085" size="1.27" layer="25" font="vector" rot="R180"/>
 <attribute name="VALUE" x="25.3365" y="16.637" size="1.27" layer="27" rot="R180"/>
@@
 <element name="R41" library="OSSI" package="R0603(1608)" value="0" x="77.7875" y="87.9475"/>
 <element name="C92" library="OSSI" package="C1210-GCM32" value="22uF,1210" x="57.4675" y="62.5475" rot="R180"/>
-<element name="L7" library="OSSI" package="LQH32CN331K23L" value="330uH" x="41.91" y="23.8125" rot="R270"/>
+<element name="L7" library="OSSI" package="LQH32CN331K23L" value="0R" x="41.91" y="23.8125" rot="R270"/>
 <element name="R14" library="OSSI" package="R0603(1608)" value="1.5k" x="58.42" y="21.59" rot="R270"/>
 <element name="R7" library="OSSI" package="R0603(1608)" value="470k" x="70.1675" y="61.9125" rot="R180"/>

Commit message: all values for tuned results are updated
Parts:
- C24: value 13pF -> 6pF
- L14: value 26nH -> 27nH
- L16: value 0 Ohm -> 7R, 3A, Ferrite bead
- R42: value TBD -> 6.2k
Changed lines of the file:
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@@
 <attribute name="VALUE" x="12.2555" y="65.3415" size="1.27" layer="27" rot="R270"/>
 </element>
-<element name="L14" library="OSSI" package="L0603(1608)" value="26nH" x="48.5775" y="42.8625" smashed="yes" rot="R180">
+<element name="L14" library="OSSI" package="L0603(1608)" value="27nH" x="48.5775" y="42.8625" smashed="yes" rot="R180">
 <attribute name="NAME" x="52.6415" y="43.561" size="1.27" layer="25" font="vector" rot="R180"/>
 <attribute name="VALUE" x="49.4665" y="44.8945" size="1.27" layer="27" rot="R180"/>
@@
 <attribute name="VALUE" x="79.0575" y="71.12" size="1.27" layer="27" rot="R90"/>
 </element>
-<element name="R42" library="OSSI" package="R0603(1608)" value="TBD" x="78.4225" y="73.66" smashed="yes" rot="R90">
+<element name="R42" library="OSSI" package="R0603(1608)" value="6.2k" x="78.4225" y="73.66" smashed="yes" rot="R90">
 <attribute name="NAME" x="80.7085" y="72.136" size="1.27" layer="25" font="vector" rot="R90"/>
 <attribute name="VALUE" x="80.4545" y="72.771" size="1.27" layer="27" rot="R90"/>
@@
 <attribute name="VALUE" x="28.067" y="11.176" size="1.27" layer="27" rot="R90"/>
 </element>
-<element name="C24" library="OSSI" package="C0603(1608)" value="13pF" x="49.53" y="40.3225" smashed="yes" rot="R270">
+<element name="C24" library="OSSI" package="C0603(1608)" value="6pF" x="49.53" y="40.3225" smashed="yes" rot="R270">
 <attribute name="NAME" x="50.546" y="39.9415" size="1.27" layer="25" font="vector"/>
 <attribute name="VALUE" x="47.498" y="41.2115" size="1.27" layer="27" rot="R270"/>
@@
 <attribute name="VALUE" x="65.151" y="45.2755" size="1.27" layer="27"/>
 </element>
-<element name="L16" library="OSSI" package="L0805(2012)" value="0 Ohm" x="59.055" y="59.53125" smashed="yes" rot="R270">
+<element name="L16" library="OSSI" package="L0805(2012)" value="7R, 3A, Ferrite bead" x="59.055" y="59.53125" smashed="yes" rot="R270">
 <attribute name="NAME" x="60.54725" y="58.801" size="1.27" layer="25" font="vector"/>
 <attribute name="VALUE" x="56.769" y="60.42025" size="1.27" layer="27" rot="R270"/>

Commit message: some library description updated
Parts:
- L2: value (none) -> DNP
- L3: value (none) -> 0R
Changed lines of the file:
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@@
 <attribute name="VALUE" x="29.0195" y="28.321" size="1.27" layer="27" rot="R90"/>
 </element>
-<element name="L3" library="OSSI" package="L0603(1608)" value="" x="19.685" y="46.99" smashed="yes" rot="R270">
+<element name="L3" library="OSSI" package="L0603(1608)" value="0R" x="19.685" y="46.99" smashed="yes" rot="R270">
 <attribute name="NAME" x="20.701" y="45.974" size="1.27" layer="25" font="vector"/>
 <attribute name="VALUE" x="17.653" y="47.879" size="1.27" layer="27" rot="R270"/>
@@
 <attribute name="VALUE" x="18.034" y="50.292" size="1.27" layer="27" rot="R180"/>
 </element>
-<element name="L2" library="OSSI" package="L0603(1608)" value="" x="17.145" y="45.72" smashed="yes" rot="R180">
+<element name="L2" library="OSSI" package="L0603(1608)" value="DNP" x="17.145" y="45.72" smashed="yes" rot="R180">
 <attribute name="NAME" x="16.129" y="46.4185" size="1.27" layer="25" font="vector" rot="R180"/>
 <attribute name="VALUE" x="18.034" y="47.752" size="1.27" layer="27" rot="R180"/>
