File: OSSIComms/OSSICommsNew/OSSICommsNew.brd (EAGLE design)
At the start: 94 x 94 mm, 188 parts, among them Q1 NX-3215, U1 MAX2640, U10 MAX6369, U11 TPS3838, U12 MAX890L, U13 MCP1700_SOT23, U2 PE4259, U3 RF5110G, U4 OPA347, U5 MAX869L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

Commit message: design file are added / missing values are added
Parts:
- C10, C15, C9: value (none) -> 56pF
- C41: value (none) -> 4.7uF
- C44: value 100uF,1210 -> 4.7uF,1210
- C45: value (none) -> 22uF
- C46: value (none) -> 100uF
- L4: value (none) -> DNP
- L6: value (none) -> 0R
- R11: value TBD -> 750R
Changed lines of the file:
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@@
 <?xml version="1.0" encoding="utf-8"?>
 <!DOCTYPE eagle SYSTEM "eagle.dtd">
-<eagle version="6.1">
+<eagle version="6.5.0">
 <drawing>
 <settings>
@@
 <layer number="14" name="Route14" color="1" fill="6" visible="no" active="no"/>
 <layer number="15" name="Route15" color="4" fill="6" visible="no" active="no"/>
-<layer number="16" name="Bottom" color="1" fill="1" visible="yes" active="yes"/>
+<layer number="16" name="Bottom" color="1" fill="1" visible="no" active="yes"/>
 <layer number="17" name="Pads" color="2" fill="1" visible="yes" active="yes"/>
 <layer number="18" name="Vias" color="2" fill="1" visible="yes" active="yes"/>
-<layer number="19" name="Unrouted" color="6" fill="1" visible="yes" active="yes"/>
+<layer number="19" name="Unrouted" color="6" fill="1" visible="no" active="yes"/>
 <layer number="20" name="Dimension" color="15" fill="1" visible="yes" active="yes"/>
 <layer number="21" name="tPlace" color="7" fill="1" visible="yes" active="yes"/>
-<layer number="22" name="bPlace" color="7" fill="1" visible="yes" active="yes"/>
+<layer number="22" name="bPlace" color="7" fill="1" visible="no" active="yes"/>
 <layer number="23" name="tOrigins" color="15" fill="1" visible="no" active="yes"/>
 <layer number="24" name="bOrigins" color="15" fill="1" visible="no" active="yes"/>
-<layer number="25" name="tNames" color="15" fill="1" visible="yes" active="yes"/>
-<layer number="26" name="bNames" color="15" fill="1" visible="yes" active="yes"/>
+<layer number="25" name="tNames" color="15" fill="1" visible="no" active="yes"/>
+<layer number="26" name="bNames" color="15" fill="1" visible="no" active="yes"/>
 <layer number="27" name="tValues" color="7" fill="1" visible="no" active="yes"/>
 <layer number="28" name="bValues" color="7" fill="1" visible="no" active="yes"/>
@@
 <layer number="50" name="dxf" color="7" fill="1" visible="no" active="no"/>
 <layer number="51" name="tDocu" color="7" fill="1" visible="yes" active="yes"/>
-<layer number="52" name="bDocu" color="7" fill="1" visible="yes" active="yes"/>
+<layer number="52" name="bDocu" color="7" fill="1" visible="no" active="yes"/>
 <layer number="53" name="tGND_GNDA" color="7" fill="9" visible="no" active="no"/>
 <layer number="54" name="bGND_GNDA" color="1" fill="9" visible="no" active="no"/>
@@
 </class>
 </classes>
-<designrules>
+<designrules name="default">
 <description language="de">&lt;b&gt;EAGLE Design Rules&lt;/b&gt;
 &lt;p&gt;
@@
 <attribute name="VALUE" x="25.3365" y="16.637" size="1.27" layer="27" rot="R180"/>
 </element>
-<element name="L6" library="OSSI" package="L0603(1608)" value="" x="17.78" y="25.4" smashed="yes" rot="R270">
+<element name="L6" library="OSSI" package="L0603(1608)" value="0R" x="17.78" y="25.4" smashed="yes" rot="R270">
 <attribute name="NAME" x="19.1135" y="24.0665" size="1.27" layer="25" font="vector"/>
 <attribute name="VALUE" x="15.748" y="26.289" size="1.27" layer="27" rot="R270"/>
 </element>
-<element name="L4" library="OSSI" package="L0603(1608)" value="" x="15.24" y="24.13" smashed="yes" rot="R180">
+<element name="L4" library="OSSI" package="L0603(1608)" value="DNP" x="15.24" y="24.13" smashed="yes" rot="R180">
 <attribute name="NAME" x="11.811" y="23.4315" size="1.27" layer="25" font="vector"/>
 <attribute name="VALUE" x="16.129" y="26.162" size="1.27" layer="27" rot="R180"/>
@@
 <attribute name="VALUE" x="67.15125" y="34.44875" size="1.27" layer="27"/>
 </element>
-<element name="C46" library="OSSI" package="C1210-GCM32" value="" x="70.32625" y="18.0975" smashed="yes">
+<element name="C46" library="OSSI" package="C1210-GCM32" value="100uF" x="70.32625" y="18.0975" smashed="yes">
 <attribute name="NAME" x="72.86625" y="17.4625" size="1.27" layer="25" font="vector"/>
 <attribute name="VALUE" x="67.15125" y="14.9225" size="1.27" layer="27"/>
 </element>
-<element name="C45" library="OSSI" package="C1210-GCM32" value="" x="70.32625" y="21.2725" smashed="yes">
+<element name="C45" library="OSSI" package="C1210-GCM32" value="22uF" x="70.32625" y="21.2725" smashed="yes">
 <attribute name="NAME" x="72.86625" y="20.6375" size="1.27" layer="25" font="vector"/>
 <attribute name="VALUE" x="67.15125" y="18.0975" size="1.27" layer="27"/>
 </element>
-<element name="C41" library="OSSI" package="C1210-GCM32" value="" x="70.32625" y="40.64" smashed="yes">
+<element name="C41" library="OSSI" package="C1210-GCM32" value="4.7uF" x="70.32625" y="40.64" smashed="yes">
 <attribute name="NAME" x="73.18375" y="40.005" size="1.27" layer="25" font="vector"/>
 <attribute name="VALUE" x="67.15125" y="37.465" size="1.27" layer="27"/>
 </element>
-<element name="C44" library="OSSI" package="C0805(2012)" value="100uF,1210" x="70.32625" y="23.97125" smashed="yes">
+<element name="C44" library="OSSI" package="C0805(2012)" value="4.7uF,1210" x="70.32625" y="23.97125" smashed="yes">
 <attribute name="NAME" x="72.29475" y="23.39975" size="1.27" layer="25" font="vector"/>
 <attribute name="VALUE" x="69.43725" y="21.68525" size="1.27" layer="27"/>
@@
 <attribute name="VALUE" x="64.262" y="28.321" size="1.27" layer="27" rot="R90"/>
 </element>
-<element name="R11" library="OSSI" package="R0603(1608)" value="TBD" x="68.58" y="47.3075" smashed="yes" rot="R270">
+<element name="R11" library="OSSI" package="R0603(1608)" value="750R" x="68.58" y="47.3075" smashed="yes" rot="R270">
 <attribute name="NAME" x="69.2785" y="48.641" size="1.27" layer="25" font="vector" rot="R90"/>
 <attribute name="VALUE" x="66.548" y="48.1965" size="1.27" layer="27" rot="R270"/>
@@
 <attribute name="VALUE" x="32.1945" y="28.321" size="1.27" layer="27" rot="R90"/>
 </element>
-<element name="C15" library="OSSI" package="C0603(1608)" value="" x="17.78" y="17.4625" smashed="yes" rot="R270">
+<element name="C15" library="OSSI" package="C0603(1608)" value="56pF" x="17.78" y="17.4625" smashed="yes" rot="R270">
 <attribute name="NAME" x="17.0815" y="16.129" size="1.27" layer="25" font="vector" rot="R270"/>
 <attribute name="VALUE" x="15.748" y="18.3515" size="1.27" layer="27" rot="R270"/>
 </element>
-<element name="C9" library="OSSI" package="C0603(1608)" value="" x="17.78" y="22.5425" smashed="yes" rot="R270">
+<element name="C9" library="OSSI" package="C0603(1608)" value="56pF" x="17.78" y="22.5425" smashed="yes" rot="R270">
 <attribute name="NAME" x="18.796" y="22.1615" size="1.27" layer="25" font="vector"/>
 <attribute name="VALUE" x="15.748" y="23.4315" size="1.27" layer="27" rot="R270"/>
@@
 <attribute name="VALUE" x="18.034" y="47.752" size="1.27" layer="27" rot="R180"/>
 </element>
-<element name="C10" library="OSSI" package="C0603(1608)" value="" x="13.0175" y="20.0025" smashed="yes">
+<element name="C10" library="OSSI" package="C0603(1608)" value="56pF" x="13.0175" y="20.0025" smashed="yes">
 <attribute name="NAME" x="12.1285" y="20.8915" size="1.27" layer="25" font="vector"/>
 <attribute name="VALUE" x="12.1285" y="17.9705" size="1.27" layer="27"/>
