File: OSSIEPS/OSSIEPSNew/OSSIEPSNew.sch (EAGLE design)
At the start: 138 parts, among them U1 LT3479, U10 LTC4411, U11 SN74LVC1T45-EP, U12 SN74LVC1T45-EP, U13 MAX890L, U14 MAX890L, U2 LT3479, U3 LT3652, U4 LTC4411, U5 LTC4411, U6 LTC4425, U7 TPS63020, U8 LTC4411, U9 LTC4411, X1 ESQ-126-38-G-D, X10 P-PAD-S, X11 P-PAD-S, X12 P-PAD-S, X13 P-PAD-S, X14 P-PAD-S, X15 P-PAD-S, X16 P-PAD-S, X17 P-PAD-S, X18 P-PAD-S, X2 DF13DF13-8P-1.25DSA, X3 DF13DF13-8P-1.25DSA, X4 DF13-10P-1.25DSA, X5 P-PAD, X6 P-PAD, X7 P-PAD, X8 E62-10K, X9 P-PAD-S

Commit message: new eps board being added
Parts:
- removed C16, C25, C26, C27: 10uF, OSSI:C1210(3225)-GCM32
- removed C17: 470pF, OSSI:C0603(1608)
- removed C18, C20, C28: 0.1uF, OSSI:C0603(1608)
- removed C19: 10nF, OSSI:C0603(1608)
- removed C21: 100pF, OSSI:C0603(1608)
- removed C31, C34: 4.7uF, 1206, OSSI:C1206(3216)-GCM31
- removed D4: STPS5L60, OSSI:STPS5L60
- removed D7, D8: PMEG6020EP, OSSI:PMEG6020EP
- removed JP1, JP10, JP2, JP5, JP6, JP8, JP9: (no value), OSSI:JP1Q
- removed JP11: (no value), SparkFun:M03POLAR
- removed L1: 1.5uH, OSSI:LXFL4020
- removed L4: 4.7uH, OSSI:LRLF7030
- removed U10, U9: LTC4411, OSSI:LTC4411
- removed U12: SN74LVC1T45-EP, OSSI:SN74LVC1T45-EP
- removed U7: TPS63020, OSSI:TPS63020
- removed X10, X11, X12, X13, X14, X15, X16, X17, X18, X9: P-PAD-S, OSSI:P-PAD-S
- removed X7: P-PAD, OSSI:P-PAD
- added TR3: FDV301N, OSSI:FDV301N
- C15: value 2.2uF -> 0.1uF; device OSSI:C1206(3216)-GCM31 -> OSSI:C0603(1608)
- C23, C24: value 10uF -> 22uF
- R11: value 17.8k -> 47k
- R12: value 4.3k -> 47k
- R13: value 169k -> 750k
- R14: value 51k -> 1.5M
- R16: value 1.2M -> 750k
- R17: value 169k -> 470k
- R18: value (none) -> 511; device OSSI:R0603(1608) -> OSSI:RWSL1206
- R19, R20, R25, R32: value 1M -> 470k
- R24: value 2.49k -> 2k
- R26: value 1.5K -> 470k
- R28: value 1M -> 47k
- R29: value 1.5K -> 1.5k
- R31: value 1M -> 20m / 10m; device OSSI:R0603(1608) -> OSSI:RWSL1206
- R37, R38: value (none) -> 1.2k
- R39: value 511k -> 511; device OSSI:R0805(2012) -> OSSI:RWSL1206
- R40: value (none) -> 1R5, 20W, 1%
- U2: value LT3479 -> MAX4376; device OSSI:LT3479 -> OSSI:MAX4376
- X2: value DF13DF13-8P-1.25DSA -> 53015-03; device OSSI:DF13DF13-8P-1.25DSA -> OSSI:53015-03
- X3: value DF13DF13-8P-1.25DSA -> 5268-02; device OSSI:DF13DF13-8P-1.25DSA -> OSSI:5268-02
- X4: value DF13-10P-1.25DSA -> 5268-02; device OSSI:DF13-10P-1.25DSA -> OSSI:5268-02
- X5: value P-PAD -> 5268-03; device OSSI:P-PAD -> OSSI:5268-03
- X6: value P-PAD -> 5268-02; device OSSI:P-PAD -> OSSI:5268-02
Connections:
- removed net N$15: L4.1, U2.P$3
- removed net N$25: C17.2, R13.1, R14.2, U2.P$11
- removed net N$26: C21.1, U2.P$10, U2.P$9
- removed net N$27: R11.2, U2.P$6
- removed net N$28: C15.1, JP1.2, JP2.1, U2.P$4, U2.P$5, U2.P$7
- removed net N$30: L1.1, U7.L1, U7.L1_2
- removed net N$32: L1.2, U7.L2, U7.L2_2
- removed net N$34: C25.1, C26.1, C27.1, JP5.1, R17.2, U7.VOUT, U7.VOUT2
- removed net N$35: R17.1, R18.2, U7.FB
- removed net N$36: C28.1, U7.SYNC/PS, U7.VINA
- removed net N$41: R28.2, R29.1, U7.EN
- removed net N$43: D8.A, JP5.2, U8.P$1
- removed net N$45: R25.2, R26.1, U6.P$6
- removed net N$47: C31.1, C34.1, D7.C, JP8.2, U10.P$5, U9.P$5, X10.P$1
- removed net N$48: R29.2, U12.P$4
- removed net N$55: JP1.1, X11.P$1
- removed net SECONDARY_SCL: X1.47, X4.7
- removed net SECONDARY_SDA: X1.49, X4.6
- removed net SUN: X1.27, X16.P$1
- new net BAT_TEMP: X1.47
- new net BUS_CS: U2.P$1, X1.27
- new net SUPERCAP_TEMP: X1.49
- net 3.3VOBC: now also C15.1, U2.P$3; no longer U12.P$1, U12.P$5, X18.P$1, X3.4, X3.5
- net ANT_COIL1: now also X2.3; no longer X5.P$1
- net ANT_COIL2: now also X2.2; no longer X6.P$1
- net ANT_DEPLOY1: now also R11.2
- net ANT_DEPLOY2: now also R12.2
- net BEACON_-FAULT: no longer X4.9
- net BEACON_OFF: no longer X4.10
- net BEACON_SCL: no longer X4.4
- net BEACON_SDA: no longer X4.3
- net GND: now also R12.1, R13.2, R17.2, R25.1, R28.1, TR3.S, U2.P$2, U6.P$4, X5.3, X6.2; no longer C16.2, C18.1, C19.1, C20.2, C21.2, C25.2, C26.2, C27.2, C28.2, C31.2, C34.2, JP10.2, JP11.3, R14.1, R18.1, U10.P$2, U10.P$3, U12.P$2, U2.P$14, U2.P$15, U2.P$16, U2.P$17, U2.P$8, U7.GND, U7.PGND, U8.P$3, U9.P$2, U9.P$3, X17.P$1, X2.3, X3.1, X3.2, X3.3, X4.5, X4.8
- net N$14: now also R13.1, R14.2, U6.P$5; no longer D8.C, U8.P$5, X9.P$1
- net N$18: now also X3.2; no longer D7.A, U10.P$1, U9.P$1, X12.P$1
- net N$20: now also R25.2, U6.P$6; no longer R26.2
- net N$21: now also C23.1, R18.1; no longer C18.2, U2.P$13
- net N$22: now also R26.1, TR3.D, U8.P$3; no longer D4.A, L4.2, U2.P$1, U2.P$2
- net N$23: now also R29.2, TR3.G; no longer C19.2, R12.1
- net N$24: now also C12.+, C13.+, C14.+, R31.1, U2.P$4, X8.C; no longer R12.2, U2.P$12
- net N$44: no longer JP2.2
- net N$46: now also X4.1; no longer JP6.1
- net N$54: now also X3.1, X8.NC; no longer JP8.1, JP9.2
- net N$57: now also X2.1; no longer X7.P$1
- net PANELTEMP_SCL: no longer X2.2
- net PANELTEMP_SDA: no longer X2.1
- net SCCHG_EN: now also R17.1
- net SCOUT_-PG: no longer R31.2, U7.PG
- net SCOUT_EN: now also R28.2, R29.1; no longer U12.P$3
- net SOLAR_CS1: no longer X2.8
- net SOLAR_CS2: no longer X2.7
- net SOLAR_CS3: no longer X2.6
- net SOLAR_CS4: no longer X2.5
- net SOLAR_CS5: no longer X2.4
- net STRUT_GND: now also H1.MOUNT; no longer H4.MOUNT
- net VBAT: now also R26.2, U8.P$1, X6.1; no longer JP10.1, X13.P$1, X14.P$1
- net VBUS: now also R31.2, U2.P$5; no longer C12.+, C13.+, C14.+, JP9.1, R31.1, X15.P$1, X4.1, X4.2
- net VMID: now also X5.2; no longer JP11.2
- net VSC_IN: now also U8.P$5; no longer C16.1, C17.1, C20.1, D4.C, R13.2, R25.1, U6.P$5
- net VSOLAR: now also X1.3, X1.4, X4.2; no longer JP6.2, X3.6, X3.7, X3.8
- net VSUPERCAP: now also R14.1, R18.2, X5.1; no longer C23.1, JP11.1, R28.1, U12.P$6, U7.VIN, U7.VIN2
Other:
- note added: "1150mA current Limit to cut the nichrome wire"
- note added: "LDO Mode"
- note added: "Power to supercap charger off by default"
- note added: "Pull Down R on both sides"
- note added: "Supercap charging OFF by Default"
- note added: "VBAT"
- note added: "Vout Set to 3.6V"
- note added: "charge current limited to 500mA"
- note added: "charge supercap when Vin > 3.6V"
- note added: "for 2.4A limit at 3.6V"
- note removed: "5.3V setting"
- note removed: "500mA charging"
- note removed: "Add Antenna Deploy signal"
- note removed: "Chage Resistor Size to 1206!!!"
- note removed: "Change to FDV301"
- note removed: "Charge Supercap by default, turned off by OBC"
- note removed: "Default???"
- note removed: "Move this to front !!!!"
- note removed: "Normal Mode"
- note removed: "Pulldown for gate??"
- note removed: "VBAT or VBUS??"
- note removed: "VINA ULVO"
- note removed: "connect with wire"
- note removed: "pullup to ?"
- moved on the sheet: C12, C13, C14, C15, C22, C23, C32, C36, D5, H1, H2, H3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

Commit message: battery supercap board added / library added
Parts:
- added TP1: TP, OSSI:TP
- X2: value 53015-03 -> 5268-03; device OSSI:53015-03 -> OSSI:5268-03
Connections:
- net GND: now also TP1.TP
Other:
- moved on the sheet: X2
Changed lines of the file:
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@@
 <part name="C36" library="OSSI" deviceset="C" device="0805(2012)"/>
 <part name="U$1" library="OSSI" deviceset="OSSILOGO" device="RECT"/>
-<part name="X2" library="OSSI" deviceset="53015-03" device=""/>
 <part name="X8" library="OSSI" deviceset="E62-10K" device=""/>
 <part name="R11" library="OSSI" deviceset="R" device="0603(1608)" value="47k"/>
@@
 <part name="X5" library="OSSI" deviceset="5268-03" device=""/>
 <part name="X6" library="OSSI" deviceset="5268-02" device=""/>
+<part name="TP1" library="OSSI" deviceset="TP" device=""/>
+<part name="X2" library="OSSI" deviceset="5268-03" device=""/>
 </parts>
 <sheets>
@@
 <instance part="GND55" gate="1" x="162.56" y="78.74"/>
 <instance part="C36" gate="G$1" x="149.86" y="88.9"/>
+<instance part="TP1" gate="G$1" x="223.52" y="127"/>
 </instances>
 <busses>
@@
 <wire x1="208.28" y1="132.08" x2="215.9" y2="132.08" width="0.1524" layer="91"/>
 <wire x1="215.9" y1="132.08" x2="215.9" y2="121.92" width="0.1524" layer="91"/>
+<pinref part="TP1" gate="G$1" pin="TP"/>
+<wire x1="223.52" y1="124.46" x2="223.52" y2="121.92" width="0.1524" layer="91"/>
+<wire x1="223.52" y1="121.92" x2="215.9" y2="121.92" width="0.1524" layer="91"/>
+<junction x="215.9" y="121.92"/>
 </segment>
 <segment>
@@
 <instance part="VBAT3" gate="G$1" x="182.88" y="160.02"/>
 <instance part="R40" gate="G$1" x="269.24" y="93.98"/>
-<instance part="X2" gate="G$1" x="302.26" y="124.46"/>
 <instance part="R11" gate="G$1" x="142.24" y="119.38" rot="R90"/>
 <instance part="R12" gate="G$1" x="142.24" y="76.2" rot="R90"/>
 <instance part="GND18" gate="1" x="142.24" y="109.22"/>
 <instance part="GND19" gate="1" x="142.24" y="66.04"/>
+<instance part="X2" gate="G$1" x="304.8" y="124.46"/>
 </instances>
 <busses>
@@
 <wire x1="289.56" y1="137.16" x2="289.56" y2="129.54" width="0.1524" layer="91"/>
 <wire x1="289.56" y1="129.54" x2="289.56" y2="127" width="0.1524" layer="91"/>
-<wire x1="289.56" y1="127" x2="297.18" y2="127" width="0.1524" layer="91"/>
+<wire x1="289.56" y1="127" x2="299.72" y2="127" width="0.1524" layer="91"/>
 <pinref part="X2" gate="G$1" pin="3"/>
 </segment>
@@
 <wire x1="281.94" y1="106.68" x2="289.56" y2="106.68" width="0.1524" layer="91"/>
 <wire x1="289.56" y1="106.68" x2="289.56" y2="124.46" width="0.1524" layer="91"/>
-<wire x1="289.56" y1="124.46" x2="297.18" y2="124.46" width="0.1524" layer="91"/>
+<wire x1="289.56" y1="124.46" x2="299.72" y2="124.46" width="0.1524" layer="91"/>
 <pinref part="X2" gate="G$1" pin="2"/>
 </segment>
@@
 <wire x1="281.94" y1="93.98" x2="292.1" y2="93.98" width="0.1524" layer="91"/>
 <wire x1="292.1" y1="93.98" x2="292.1" y2="121.92" width="0.1524" layer="91"/>
-<wire x1="292.1" y1="121.92" x2="297.18" y2="121.92" width="0.1524" layer="91"/>
+<wire x1="292.1" y1="121.92" x2="299.72" y2="121.92" width="0.1524" layer="91"/>
 <pinref part="X2" gate="G$1" pin="1"/>
 </segment>

Commit message: schematics renumbered
Parts:
- removed C29, C30: 100nF, 0805, OSSI:C0805(2012)
- removed C32, C33: 4.7uF, 1206, OSSI:C1206(3216)-GCM31
- removed C35: (no value), OSSI:C0603(1608)
- removed C36: (no value), OSSI:C0805(2012)
- removed D6: PMEG6020EP, OSSI:PMEG6020EP
- removed L3: 10uH, OSSI:LRLF12545
- removed U11: SN74LVC1T45-EP, OSSI:SN74LVC1T45-EP
- removed U13, U14: MAX890L, OSSI:MAX890L
- removed X8: E62-10K, OSSI:E62-10K
- added C16: 100uF, OSSI:C1210(3225)-TMK325
- added C17, C21: 10uF, OSSI:C1210(3225)-GCM32
- added C18: 10nF, OSSI:C0603(1608)
- added C19: 470pF, OSSI:C0603(1608)
- added C20: 0.1uF, OSSI:C0603(1608)
- added D4: PMEG6020EP, OSSI:PMEG6020EP
- added L1: 4.7uH, OSSI:LRLF7030
- added U10, U7: LTC4411, OSSI:LTC4411
- added U9: MAX4376, OSSI:MAX4376
- added X7: 5268-02, OSSI:5268-02
- C1: value 2.2uF -> (none); device OSSI:C1206(3216)-GCM31 -> OSSI:C0805(2012)
- C10: value 1uF, 100V -> 0 Ohm; device OSSI:C0805(2012) -> OSSI:C0603(1608)
- C11: value 0 Ohm -> (none)
- C2, C3: value 10uF -> 100nF, 0805; device OSSI:C1210(3225)-GCM32 -> OSSI:C0805(2012)
- C22: value 2.2uF -> 1uF, 100V; device OSSI:C1206(3216)-GCM31 -> OSSI:C0805(2012)
- C23: value 22uF -> 0.1uF; device OSSI:C1210(3225)-GCM32 -> OSSI:C0603(1608)
- C24: value 22uF -> 4.7uF, 1206; device OSSI:C1210(3225)-GCM32 -> OSSI:C1206(3216)-GCM31
- C4: value 100uF -> 2.2uF; device OSSI:C1210(3225)-TMK325 -> OSSI:C1206(3216)-GCM31
- C5: value 470pF -> 22uF; device OSSI:C0603(1608) -> OSSI:C1210(3225)-GCM32
- C6: value 0.1uF -> 22uF; device OSSI:C0603(1608) -> OSSI:C1210(3225)-GCM32
- C7: value 10nF -> 100pF
- C8: value 0.1uF -> 2.2uF; device OSSI:C0603(1608) -> OSSI:C1206(3216)-GCM31
- C9: value 100pF -> 4.7uF, 1206; device OSSI:C0603(1608) -> OSSI:C1206(3216)-GCM31
- D1: value STPS5L60 -> PMEG6020EP; device OSSI:STPS5L60 -> OSSI:PMEG6020EP
- D3: value PMEG6020EP -> STPS5L60; device OSSI:PMEG6020EP -> OSSI:STPS5L60
- L2: value 4.7uH -> 10uH; device OSSI:LRLF7030 -> OSSI:LRLF12545
- R1: value 17.8k -> 511; device OSSI:R0603(1608) -> OSSI:RWSL1206
- R10: value 0.1 -> 100k; device OSSI:RWSL1206 -> OSSI:R0603(1608)
- R12: value 47k -> 1.5k
- R13: value 750k -> 470k
- R14: value 1.5M -> 511; device OSSI:R0603(1608) -> OSSI:RWSL1206
- R15: value 1.5M -> 470k
- R17, R20, R30: value 470k -> 1.5M
- R18: value 511 -> 2k; device OSSI:RWSL1206 -> OSSI:R0603(1608)
- R2: value 4.3k -> 47k
- R21: value 470k -> 750k
- R22: value 200k -> 470k
- R23: value 100k -> 470k
- R24: value 2k -> 17.8k
- R25: value 470k -> 30.9k
- R26: value 470k -> 0.1; device OSSI:R0603(1608) -> OSSI:RWSL1206
- R27: value 470k -> 169k
- R28: value 47k -> 100k
- R29: value 1.5k -> 100k
- R3: value 169k -> 1.5k
- R31: value 20m / 10m -> 4.3k; device OSSI:RWSL1206 -> OSSI:R0603(1608)
- R32: value 470k -> 300k
- R33: value 1.5k -> 200k
- R34: value 1.5k -> 36k
- R35: value 100k -> 20m / 10m; device OSSI:R0603(1608) -> OSSI:RWSL1206
- R36: value 100k -> 0.05; device OSSI:R0603(1608) -> OSSI:RWSL1206
- R37, R38: value 1.2k -> 470k
- R39: value 511 -> 470k; device OSSI:RWSL1206 -> OSSI:R0603(1608)
- R4: value 30.9k -> 1.2k
- R40: value 1R5, 20W, 1% -> 470k; device OSSI:RPWR263S -> OSSI:R0603(1608)
- R5: value 300k -> 1R5, 20W, 1%; device OSSI:R0603(1608) -> OSSI:RPWR263S
- R6: value 1.5M -> 47k
- R7: value 36k -> 1.2k
- R8: value 100k -> 1.5k
- R9: value 0.05 -> 100k; device OSSI:RWSL1206 -> OSSI:R0603(1608)
- U1: value LT3479 -> MAX890L; device OSSI:LT3479 -> OSSI:MAX890L
- U2: value MAX4376 -> MAX890L; device OSSI:MAX4376 -> OSSI:MAX890L
- U3: value LT3652 -> LTC4411; device OSSI:LT3652 -> OSSI:LTC4411
- U4: value LTC4411 -> LTC4425; device OSSI:LTC4411 -> OSSI:LTC4425
- U5: value LTC4411 -> SN74LVC1T45-EP; device OSSI:LTC4411 -> OSSI:SN74LVC1T45-EP
- U6: value LTC4425 -> LT3479; device OSSI:LTC4425 -> OSSI:LT3479
- U8: value LTC4411 -> LT3652; device OSSI:LTC4411 -> OSSI:LT3652
- X3: value 5268-02 -> 5268-03; device OSSI:5268-02 -> OSSI:5268-03
- X5: value 5268-03 -> 5268-02; device OSSI:5268-03 -> OSSI:5268-02
- X6: value 5268-02 -> E62-10K; device OSSI:5268-02 -> OSSI:E62-10K
- renumbered JP4 to JP1, JP7 to JP2
Connections:
- net 3.3VOBC: now also C23.1, U5.P$1, U5.P$5, U9.P$3; no longer C15.1, U11.P$1, U11.P$5, U2.P$3
- net ANT_COIL1: now also C3.1, U2.P$6, U2.P$7; no longer C29.1, U13.P$6, U13.P$7
- net ANT_COIL2: now also C2.1, U1.P$6, U1.P$7; no longer C30.1, U14.P$6, U14.P$7
- net ANT_DEPLOY1: now also R6.2, R8.1; no longer R11.2, R33.1
- net ANT_DEPLOY2: now also R2.2, R3.1; no longer R12.2, R34.1
- net BAT_-CHRG: now also R39.1, U8.P$4; no longer R19.1, U3.P$4
- net BAT_-FAULT: now also R38.1, U8.P$5; no longer R20.1, U3.P$5
- net BAT_-ON: now also R37.1, U7.P$4; no longer R27.1, U5.P$4
- net BUS_CS: now also U9.P$1; no longer U2.P$1
- net GND: now also C10.2, C15.1, C17.2, C18.1, C20.2, C21.2, C4.2, C5.2, C6.2, C7.2, D3.A, R16.2, R18.1, R2.1, R22.1, R23.2, R26.2, R29.1, R30.1, R5.1, R7.1, U1.P$4, U10.P$2, U10.P$3, U2.P$4, U3.P$2, U4.P$13, U4.P$4, U6.P$14, U6.P$15, U6.P$16, U6.P$17, U6.P$8, U7.P$2, U7.P$3, U8.P$13, U9.P$2, X3.3, X4.2; no longer C15.2, C22.2, C29.2, C30.2, C32.2, C33.2, C35.2, C36.2, C6.1, C7.1, D2.A, R10.2, R12.1, R13.2, R17.2, R23.1, R37.1, R38.1, R39.1, R40.1, R8.1, U1.P$14, U1.P$15, U1.P$16, U1.P$17, U1.P$8, U11.P$2, U13.P$4, U14.P$4, U2.P$2, U3.P$13, U4.P$2, U4.P$3, U5.P$3, U6.P$13, U6.P$4, U8.P$2, X5.3, X6.2
- net N$1: now also L1.1, U6.P$3; no longer L2.1, U1.P$3
- net N$10: now also C7.1, U6.P$10, U6.P$9; no longer C9.1, U1.P$10, U1.P$9
- net N$11: now also R24.2, U6.P$6; no longer R1.2, U1.P$6
- net N$12: now also R28.2, R33.1, U8.P$3; no longer R22.1, R23.2, U3.P$3
- net N$13: now also C22.2, D1.C, U8.P$11; no longer C10.2, D3.C, U3.P$11
- net N$14: now also R16.1, R20.2, U4.P$5; no longer R13.1, R14.2, U6.P$5
- net N$16: now also C22.1, D3.C, L2.1, U8.P$12; no longer C10.1, D2.C, L3.1, U3.P$12
- net N$17: now also R30.2, R32.1, U8.P$7; no longer R5.1, R6.2, U3.P$7
- net N$18: now also C24.1, C9.1, D4.C, U10.P$5, U7.P$5, X5.2; no longer C32.1, C33.1, D6.C, U4.P$5, U5.P$5, X3.2
- net N$19: now also C10.1, U8.P$6; no longer C11.1, U3.P$6
- net N$2: now also R29.2, R34.1, U8.P$2; no longer R7.1, R8.2, U3.P$2
- net N$20: now also R22.2, U4.P$6, U5.P$4; no longer R25.2, U11.P$4, U6.P$6
- net N$21: now also C5.1, R14.1; no longer C23.1, R18.1
- net N$22: now also R13.1, U3.P$3; no longer R26.1, U8.P$3
- net N$23: now also R12.2; no longer R29.2
- net N$24: now also R35.1, U9.P$4, X6.C; no longer R31.1, U2.P$4, X8.C
- net N$29: now also R17.2, R21.1, U4.P$9; no longer R15.2, R16.1, U6.P$9
- net N$3: now also C19.1, C20.1, C21.1, D2.C, R27.2, U8.P$1; no longer C2.1, C5.1, C8.1, D1.C, R3.2, U3.P$1
- net N$31: now also R21.2, U4.P$7; no longer R16.2, U6.P$7
- net N$33: now also R3.2, TR1.G; no longer R34.2, TR2.G
- net N$37: now also U2.P$8; no longer U13.P$8
- net N$38: now also U1.P$8; no longer U14.P$8
- net N$39: now also D5.A, U10.P$1; no longer D6.A, U4.P$1
- net N$4: now also C16.2, R26.1; no longer C4.2, R10.1
- net N$40: now also R18.2, U4.P$3; no longer R24.2, U6.P$3
- net N$42: now also D4.A, U7.P$1; no longer D5.A, U5.P$1
- net N$44: now also C8.1, R33.2, R34.2, U6.P$4, U6.P$5, U6.P$7; no longer C1.1, R22.2, R7.2, U1.P$4, U1.P$5, U1.P$7
- net N$46: now also X7.1; no longer X4.1
- net N$49: now also R8.2, TR2.G; no longer R33.2, TR1.G
- net N$5: now also C15.2, U6.P$13; no longer C6.2, U1.P$13
- net N$50: now also R9.1, TR2.D, U2.P$3; no longer R35.1, TR1.D, U13.P$3
- net N$51: now also R10.1, TR1.D, U1.P$3; no longer R36.1, TR2.D, U14.P$3
- net N$52: now also R7.2, U2.P$5; no longer R37.2, U13.P$5
- net N$53: now also R4.2, U1.P$5; no longer R38.2, U14.P$5
- net N$54: now also X5.1, X6.NC; no longer X3.1, X8.NC
- net N$57: now also R5.2; no longer R40.2
- net N$6: now also D2.A, L1.2, U6.P$1, U6.P$2; no longer D1.A, L2.2, U1.P$1, U1.P$2
- net N$7: now also C18.2, R31.1; no longer C7.2, R2.1
- net N$8: now also R31.2, U6.P$12; no longer R2.2, U1.P$12
- net N$9: now also C19.2, R25.2, R27.1, U6.P$11; no longer C5.2, R3.1, R4.2, U1.P$11
- net SCCHG_EN: now also R23.1, U5.P$3; no longer R17.1, U11.P$3
- net SCOUT_EN: now also R11.2, R12.1; no longer R28.2, R29.1
- net SC_-ON: now also R15.1, U3.P$4; no longer R30.1, U8.P$4
- net SC_-PFO: now also R19.2, U4.P$8; no longer R32.2, U6.P$8
- net SENSE: now also L2.2, R36.1, U8.P$10; no longer L3.2, R9.1, U3.P$10
- net SOLAR_-ON: now also R40.1, U10.P$4; no longer R21.1, U4.P$4
- net STRUT_GND: now also C1.1, H4.MOUNT, R1.2; no longer C36.1, H1.MOUNT, R39.2
- net VBAT: now also C11.1, C16.1, C17.1, D1.A, R10.2, R13.2, R32.2, U1.P$1, U1.P$2, U2.P$1, U2.P$2, U3.P$1, U8.P$9, X4.1; no longer C3.1, C35.1, C4.1, D3.A, R26.2, R35.2, R5.2, U13.P$1, U13.P$2, U14.P$1, U14.P$2, U3.P$9, U8.P$1, X6.1
- net VBUS: now also R15.2, R19.1, R35.2, R37.2, R38.2, R39.2, R40.2, U9.P$5; no longer R19.2, R20.2, R21.2, R27.2, R30.2, R31.2, R32.1, U2.P$5
- net VMID: now also U4.P$10, X3.2; no longer U6.P$10, X5.2
- net VSC_IN: now also C4.1, R17.1, U3.P$5, U4.P$11, U4.P$12, U5.P$6; no longer C22.1, R15.1, U11.P$6, U6.P$11, U6.P$12, U8.P$5
- net VSOLAR: now also X7.2; no longer X4.2
- net VSUPERCAP: now also C6.1, R14.2, R20.1, U4.P$1, U4.P$2, X3.1; no longer C24.1, R14.1, R18.2, U6.P$1, U6.P$2, X5.1
