File: OSSIEPS/OSSIEPSNew/OSSIEPSNew.sch (EAGLE design)
At the start: 100 parts, among them U1 MAX890L, U10 LTC4411, U2 MAX890L, U3 LTC4411, U4 LTC4425, U5 SN74LVC1T45-EP, U6 LT3479, U7 LTC4411, U8 LT3652, U9 MAX4376, X1 ESQ-126-38-G-D, X2 5268-03, X3 5268-03, X4 5268-02, X5 5268-02, X6 E62-10K, X7 5268-02

Commit message: all values for tuned results are updated
Parts:
- added R41, R42: 1M, OSSI:R0603(1608)
- C1: value (none) -> 100nF
- C11: value (none) -> 22nF
- C2, C3: value 100nF, 0805 -> 1uF, 0805
- C22: value 1uF, 100V -> 1uF, 100V, 1206
- D4, D5: value PMEG6020EP -> PMEG3050BEP
- R11, R2, R6: value 47k -> 100k
- R35: value 20m / 10m -> 10m
Connections:
- net ANT_COIL1: now also R41.2
- net ANT_COIL2: now also R42.2
- net GND: now also R41.1, R42.1
Other:
- note added: "1M pulldown added!!!"
- note added: "30K added"
- note added: "To make sure OUT is zero"
Changed lines of the file:
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@@
 <part name="R36" library="OSSI" deviceset="R" device="WSL1206" value="0.05"/>
 <part name="R26" library="OSSI" deviceset="R" device="WSL1206" value="0.1"/>
-<part name="C22" library="OSSI" deviceset="C" device="0805(2012)" value="1uF, 100V"/>
+<part name="C22" library="OSSI" deviceset="C" device="0805(2012)" value="1uF, 100V, 1206"/>
 <part name="GND10" library="OSSI" deviceset="GND" device=""/>
 <part name="C10" library="OSSI" deviceset="C" device="0603(1608)" value="0 Ohm"/>
@@
 <part name="TR2" library="OSSI" deviceset="FDV301N" device=""/>
 <part name="GND47" library="OSSI" deviceset="GND" device=""/>
-<part name="C3" library="OSSI" deviceset="C" device="0805(2012)" value="100nF, 0805"/>
-<part name="C2" library="OSSI" deviceset="C" device="0805(2012)" value="100nF, 0805"/>
+<part name="C3" library="OSSI" deviceset="C" device="0805(2012)" value="1uF, 0805"/>
+<part name="C2" library="OSSI" deviceset="C" device="0805(2012)" value="1uF, 0805"/>
 <part name="GND36" library="OSSI" deviceset="GND" device=""/>
 <part name="GND48" library="OSSI" deviceset="GND" device=""/>
 <part name="STRUT_GND1" library="OSSI" deviceset="STRUT_GND" device=""/>
-<part name="D4" library="OSSI" deviceset="PMEG6020EP" device=""/>
-<part name="D5" library="OSSI" deviceset="PMEG6020EP" device=""/>
+<part name="D4" library="OSSI" deviceset="PMEG6020EP" device="" value="PMEG3050BEP"/>
+<part name="D5" library="OSSI" deviceset="PMEG6020EP" device="" value="PMEG3050BEP"/>
 <part name="C9" library="OSSI" deviceset="C" device="1206(3216)-GCM31" value="4.7uF, 1206"/>
 <part name="C24" library="OSSI" deviceset="C" device="1206(3216)-GCM31" value="4.7uF, 1206"/>
@@
 <part name="GND50" library="OSSI" deviceset="GND" device=""/>
 <part name="VBAT3" library="OSSI" deviceset="VBAT" device=""/>
-<part name="C11" library="OSSI" deviceset="C" device="0603(1608)"/>
+<part name="C11" library="OSSI" deviceset="C" device="0603(1608)" value="22nF"/>
 <part name="GND46" library="OSSI" deviceset="GND" device=""/>
 <part name="GND54" library="OSSI" deviceset="GND" device=""/>
@@
 <part name="GND55" library="OSSI" deviceset="GND" device=""/>
 <part name="R5" library="OSSI" deviceset="R" device="PWR263S" value="1R5, 20W, 1%"/>
-<part name="C1" library="OSSI" deviceset="C" device="0805(2012)"/>
+<part name="C1" library="OSSI" deviceset="C" device="0805(2012)" value="100nF"/>
 <part name="U$1" library="OSSI" deviceset="OSSILOGO" device="RECT"/>
 <part name="X6" library="OSSI" deviceset="E62-10K" device=""/>
-<part name="R6" library="OSSI" deviceset="R" device="0603(1608)" value="47k"/>
-<part name="R2" library="OSSI" deviceset="R" device="0603(1608)" value="47k"/>
+<part name="R6" library="OSSI" deviceset="R" device="0603(1608)" value="100k"/>
+<part name="R2" library="OSSI" deviceset="R" device="0603(1608)" value="100k"/>
 <part name="GND18" library="OSSI" deviceset="GND" device=""/>
 <part name="GND19" library="OSSI" deviceset="GND" device=""/>
@@
 <part name="TR3" library="OSSI" deviceset="FDV301N" device=""/>
 <part name="GND25" library="OSSI" deviceset="GND" device=""/>
-<part name="R11" library="OSSI" deviceset="R" device="0603(1608)" value="47k"/>
+<part name="R11" library="OSSI" deviceset="R" device="0603(1608)" value="100k"/>
 <part name="R12" library="OSSI" deviceset="R" device="0603(1608)" value="1.5k"/>
 <part name="GND26" library="OSSI" deviceset="GND" device=""/>
-<part name="R35" library="OSSI" deviceset="R" device="WSL1206" value="20m / 10m"/>
+<part name="R35" library="OSSI" deviceset="R" device="WSL1206" value="10m"/>
 <part name="U9" library="OSSI" deviceset="MAX4376" device=""/>
 <part name="GND27" library="OSSI" deviceset="GND" device=""/>
@@
 <part name="TP1" library="OSSI" deviceset="TP" device=""/>
 <part name="X2" library="OSSI" deviceset="5268-03" device=""/>
+<part name="R41" library="OSSI" deviceset="R" device="0603(1608)" value="1M"/>
+<part name="R42" library="OSSI" deviceset="R" device="0603(1608)" value="1M"/>
 </parts>
 <sheets>
@@
 <text x="226.06" y="81.28" size="1.778" layer="94">1150mA current Limit to cut the nichrome wire</text>
 <text x="287.02" y="86.36" size="1.778" layer="94">for 2.4A limit at 3.6V</text>
+<text x="261.62" y="129.54" size="1.778" layer="94">1M pulldown added!!!</text>
+<text x="261.62" y="101.6" size="1.778" layer="94">1M pulldown added!!!</text>
+<text x="261.62" y="127" size="1.778" layer="94">To make sure OUT is zero</text>
+<text x="261.62" y="99.06" size="1.778" layer="94">To make sure OUT is zero</text>
 </plain>
 <instances>
@@
 <instance part="GND19" gate="1" x="142.24" y="66.04"/>
 <instance part="X2" gate="G$1" x="304.8" y="124.46"/>
+<instance part="R41" gate="G$1" x="256.54" y="132.08" rot="R90"/>
+<instance part="R42" gate="G$1" x="256.54" y="101.6" rot="R90"/>
 </instances>
 <busses>
@@
 <pinref part="C3" gate="G$1" pin="2"/>
 <wire x1="243.84" y1="124.46" x2="243.84" y2="127" width="0.1524" layer="91"/>
+<pinref part="R41" gate="G$1" pin="1"/>
+<wire x1="256.54" y1="127" x2="256.54" y2="124.46" width="0.1524" layer="91"/>
+<wire x1="256.54" y1="124.46" x2="243.84" y2="124.46" width="0.1524" layer="91"/>
+<junction x="243.84" y="124.46"/>
 </segment>
 <segment>
@@
 <wire x1="243.84" y1="93.98" x2="243.84" y2="96.52" width="0.1524" layer="91"/>
 <pinref part="R5" gate="G$1" pin="1"/>
-<wire x1="264.16" y1="93.98" x2="243.84" y2="93.98" width="0.1524" layer="91"/>
+<wire x1="264.16" y1="93.98" x2="256.54" y2="93.98" width="0.1524" layer="91"/>
 <junction x="243.84" y="93.98"/>
+<pinref part="R42" gate="G$1" pin="1"/>
+<wire x1="256.54" y1="93.98" x2="243.84" y2="93.98" width="0.1524" layer="91"/>
+<wire x1="256.54" y1="93.98" x2="256.54" y2="96.52" width="0.1524" layer="91"/>
+<junction x="256.54" y="93.98"/>
 </segment>
 <segment>
@@
 <wire x1="243.84" y1="134.62" x2="243.84" y2="137.16" width="0.1524" layer="91"/>
 <junction x="243.84" y="137.16"/>
-<wire x1="243.84" y1="137.16" x2="281.94" y2="137.16" width="0.1524" layer="91"/>
+<wire x1="243.84" y1="137.16" x2="256.54" y2="137.16" width="0.1524" layer="91"/>
+<wire x1="256.54" y1="137.16" x2="281.94" y2="137.16" width="0.1524" layer="91"/>
 <wire x1="281.94" y1="137.16" x2="289.56" y2="137.16" width="0.1524" layer="91"/>
 <wire x1="289.56" y1="137.16" x2="289.56" y2="129.54" width="0.1524" layer="91"/>
@@
 <wire x1="289.56" y1="127" x2="299.72" y2="127" width="0.1524" layer="91"/>
 <pinref part="X2" gate="G$1" pin="3"/>
+<pinref part="R41" gate="G$1" pin="2"/>
+<junction x="256.54" y="137.16"/>
 </segment>
 </net>
@@
 <wire x1="243.84" y1="104.14" x2="243.84" y2="106.68" width="0.1524" layer="91"/>
 <junction x="243.84" y="106.68"/>
-<wire x1="243.84" y1="106.68" x2="281.94" y2="106.68" width="0.1524" layer="91"/>
+<wire x1="243.84" y1="106.68" x2="256.54" y2="106.68" width="0.1524" layer="91"/>
+<wire x1="256.54" y1="106.68" x2="281.94" y2="106.68" width="0.1524" layer="91"/>
 <wire x1="281.94" y1="106.68" x2="289.56" y2="106.68" width="0.1524" layer="91"/>
 <wire x1="289.56" y1="106.68" x2="289.56" y2="124.46" width="0.1524" layer="91"/>
 <wire x1="289.56" y1="124.46" x2="299.72" y2="124.46" width="0.1524" layer="91"/>
 <pinref part="X2" gate="G$1" pin="2"/>
+<pinref part="R42" gate="G$1" pin="2"/>
+<junction x="256.54" y="106.68"/>
 </segment>
 </net>
@@
 <text x="129.54" y="119.38" size="1.778" layer="94">charge supercap when Vin &gt; 3.6V</text>
 <text x="104.14" y="68.58" size="1.778" layer="94">Power to supercap charger off by default</text>
+<text x="114.3" y="149.86" size="1.778" layer="94">30K added</text>
 </plain>
 <instances>

Commit message: design flies are added
Other:
- note added: "Chassis ( Satellite Sturucture ) is conneced only to EPS module to prevent the loop path and via resistor and capacitor to protect ESD when the chassis is touched."
- note added: "For measuring currents but normally soldered"
- note added: "This setup will make sure that antennae are deployed"
- note added: "pull downs are needed to prevent the FET from fault turn on"
- note added: "pull ups are needed to prevent the MAX890 from fault turn on"
- note added: "we set the current value to cut the nichrome wire not ony cut the fishing wire"
Changed lines of the file:
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@@
 <?xml version="1.0" encoding="utf-8"?>
 <!DOCTYPE eagle SYSTEM "eagle.dtd">
-<eagle version="6.1">
+<eagle version="6.5.0">
 <drawing>
 <settings>
@@
 <sheet>
 <plain>
+<text x="111.76" y="101.6" size="1.778" layer="94">Chassis ( Satellite Sturucture ) is conneced only to EPS module to prevent the loop path and via resistor and capacitor to protect ESD when the chassis is touched.</text>
 </plain>
 <instances>
@@
 <text x="261.62" y="127" size="1.778" layer="94">To make sure OUT is zero</text>
 <text x="261.62" y="99.06" size="1.778" layer="94">To make sure OUT is zero</text>
+<text x="83.82" y="101.6" size="1.778" layer="94">pull downs are needed to prevent the FET from fault turn on</text>
+<text x="162.56" y="167.64" size="1.778" layer="94">pull ups are needed to prevent the MAX890 from fault turn on</text>
+<text x="243.84" y="154.94" size="1.778" layer="94">we set the current value to cut the nichrome wire not ony cut the fishing wire</text>
+<text x="243.84" y="152.4" size="1.778" layer="94">This setup will make sure that antennae are deployed</text>
 </plain>
 <instances>
@@
 <text x="104.14" y="68.58" size="1.778" layer="94">Power to supercap charger off by default</text>
 <text x="114.3" y="149.86" size="1.778" layer="94">30K added</text>
+<text x="40.64" y="231.14" size="1.778" layer="94">For measuring currents but normally soldered </text>
+<text x="30.48" y="205.74" size="1.778" layer="94">For measuring currents but normally soldered </text>
+<text x="233.68" y="195.58" size="1.778" layer="94" rot="R90">For measuring currents but normally soldered </text>
 </plain>
 <instances>
@@
 <pinref part="U8" gate="G$1" pin="P$5"/>
 <wire x1="157.48" y1="180.34" x2="152.4" y2="180.34" width="0.1524" layer="91"/>
-<label x="149.86" y="180.34" size="1.778" layer="95" rot="R180" xref="yes"/>
+<label x="149.86" y="180.34" size="1.778" layer="95" rot="R270" xref="yes"/>
 <pinref part="R38" gate="G$1" pin="1"/>
 <wire x1="152.4" y1="180.34" x2="149.86" y2="180.34" width="0.1524" layer="91"/>
@@
 <segment>
 <pinref part="U9" gate="G$1" pin="P$1"/>
-<wire x1="375.92" y1="205.74" x2="375.92" y2="210.82" width="0.1524" layer="91"/>
-<label x="375.92" y="210.82" size="1.778" layer="95" rot="R90" xref="yes"/>
-</segment>
-</net>
+<wire x1="375.92" y1="205.74" x2="375.92" y2="220.98" width="0.1524" layer="91"/>
+<label x="375.92" y="220.98" size="1.778" layer="95" rot="R90" xref="yes"/>
+</segment>
+</net>
