File: OSSILEDController/OSSILEDControllerNew/OSSILEDControllerNew.brd (EAGLE design)
At the start: 94 x 88 mm, 80 parts, among them Q1 NX-3215, U1 MSP430F2132, U2 OPA2347, U3 MAX4376, U4 LM7321, U5 MAX1682, U6 TPS3838, U7 MAX890L, U8 MCP1700_SOT23, X1 ESQ-126-38-G-D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

Commit message: all values for tuned results are updated
Parts:
- C11: value 1206 Cap -> 4.7uF, 1206 Cap
- R11: value 9.1k -> 5.1k
- R23: value 100k -> 1k
- R9: value 6.2k -> 3k
Changed lines of the file:
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@@
 <attribute name="VALUE" x="21.463" y="36.449" size="1.27" layer="27" rot="R270"/>
 </element>
-<element name="R23" library="OSSI" package="R0603(1608)" value="100k" x="51.435" y="33.655" smashed="yes" rot="R90">
+<element name="R23" library="OSSI" package="R0603(1608)" value="1k" x="51.435" y="33.655" smashed="yes" rot="R90">
 <attribute name="NAME" x="53.721" y="31.8135" size="1.27" layer="25" font="vector" rot="R90"/>
 <attribute name="VALUE" x="53.467" y="32.766" size="1.27" layer="27" rot="R90"/>
@@
 <attribute name="VALUE" x="60.579" y="32.131" size="1.27" layer="27" rot="R180"/>
 </element>
-<element name="C11" library="OSSI" package="C1206-GCM31" value="1206 Cap" x="56.1975" y="34.29" smashed="yes" rot="R90">
+<element name="C11" library="OSSI" package="C1206-GCM31" value="4.7uF, 1206 Cap" x="56.1975" y="34.29" smashed="yes" rot="R90">
 <attribute name="NAME" x="56.8325" y="36.83" size="1.27" layer="25" font="vector" rot="R90"/>
 <attribute name="VALUE" x="58.7375" y="31.115" size="1.27" layer="27" rot="R90"/>
@@
 <attribute name="VALUE" x="45.085" y="35.56" size="1.27" layer="27" rot="R270"/>
 </element>
-<element name="R11" library="OSSI" package="R0603(1608)" value="9.1k" x="44.45" y="34.925" smashed="yes" rot="R270">
+<element name="R11" library="OSSI" package="R0603(1608)" value="5.1k" x="44.45" y="34.925" smashed="yes" rot="R270">
 <attribute name="NAME" x="42.6085" y="36.449" size="1.27" layer="25" font="vector"/>
 <attribute name="VALUE" x="42.418" y="35.814" size="1.27" layer="27" rot="R270"/>
 </element>
-<element name="R9" library="OSSI" package="R0603(1608)" value="6.2k" x="44.45" y="32.385" smashed="yes" rot="R270">
+<element name="R9" library="OSSI" package="R0603(1608)" value="3k" x="44.45" y="32.385" smashed="yes" rot="R270">
 <attribute name="NAME" x="43.2435" y="29.464" size="1.27" layer="25" font="vector"/>
 <attribute name="VALUE" x="42.418" y="33.274" size="1.27" layer="27" rot="R270"/>

Commit message: led sch updated / design files are added
Parts:
- C1, R25: value (none) -> DNP
- R1: value 511 -> DNP
- R19: value 2.2k -> 2.4k
- moved R19 6.84 mm to (44.5, 27.9), turned to 180 degrees
Connections:
- net 3.3VLED: now also C15.1, R19.2, U5.4
- net GND: no longer R19.1
- net N$14: no longer R19.2
- net N$18: now also R19.1
- net VSUPERCAP: no longer C15.1, U5.4
Routing:
- net 3.3VLED: track 226.5 -> 261.4 mm, vias 2 -> 4
- net VSUPERCAP: track 89.2 -> 70.5 mm
- net N$18: track 2.70 -> 4.53 mm
