File: OSSIInterfaceBoard/OSSIICBNew/OSSIICBNew.sch (EAGLE design)
At the start: 24 parts, among them X1 ESQ-126-38-G-D, X3 DF13DF13A-8P-1.25H, X4 DF13DF13-8P-1.25DSA, X6 DF13DF13A-8P-1.25H, X7 DF13DF13A-8P-1.25H, X8 DF13DF13A-8P-1.25H

Commit message: design files are added
Parts:
- C43: value (none) -> DNP
- R39: value 511 -> DNP
Other:
- moved on the sheet: H3
Changed lines of the file:
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@@
 <?xml version="1.0" encoding="utf-8"?>
 <!DOCTYPE eagle SYSTEM "eagle.dtd">
-<eagle version="6.1">
+<eagle version="6.5.0">
 <drawing>
 <settings>
@@
 <part name="VSOLAR7" library="OSSI" deviceset="VSOLAR" device=""/>
 <part name="STRUT_GND2" library="OSSI" deviceset="STRUT_GND" device=""/>
-<part name="R39" library="OSSI" deviceset="R" device="WSL1206" value="511"/>
-<part name="C43" library="OSSI" deviceset="C" device="0805(2012)"/>
+<part name="R39" library="OSSI" deviceset="R" device="WSL1206" value="DNP"/>
+<part name="C43" library="OSSI" deviceset="C" device="0805(2012)" value="DNP"/>
 <part name="GND37" library="OSSI" deviceset="GND" device=""/>
 <part name="U$1" library="OSSI" deviceset="OSSILOGO" device="-10"/>
@@
 <instance part="H1" gate="G$1" x="129.54" y="66.04"/>
 <instance part="H2" gate="G$1" x="129.54" y="55.88"/>
-<instance part="H3" gate="G$1" x="144.78" y="66.04"/>
+<instance part="H3" gate="G$1" x="165.1" y="66.04"/>
 <instance part="H4" gate="G$1" x="144.78" y="43.18"/>
 <instance part="FRAME1" gate="G$1" x="0" y="0"/>
