File: BatterySuperCapBoard/BatterySuperCapBoard/BatterySuperCapBoard.brd (EAGLE design)
At the start: 94 x 88 mm, 20 parts, among them X1 ESQ-126-38-G-D, X2 WEIDMULLER

Commit message: beta 1 release
Parts:
- moved X2 8.35 mm to (72.5, 73.1)
Other:
- outline, holes or cut-outs redrawn
Changed lines of the file:
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@@
 <layer number="27" name="tValues" color="7" fill="1" visible="no" active="yes"/>
 <layer number="28" name="bValues" color="7" fill="1" visible="no" active="yes"/>
-<layer number="29" name="tStop" color="7" fill="3" visible="yes" active="yes"/>
-<layer number="30" name="bStop" color="7" fill="6" visible="yes" active="yes"/>
+<layer number="29" name="tStop" color="7" fill="3" visible="no" active="yes"/>
+<layer number="30" name="bStop" color="7" fill="6" visible="no" active="yes"/>
 <layer number="31" name="tCream" color="7" fill="4" visible="no" active="yes"/>
 <layer number="32" name="bCream" color="7" fill="5" visible="no" active="yes"/>
@@
 <board>
 <plain>
-<wire x1="91" y1="0" x2="54.5" y2="0" width="0" layer="20"/>
-<wire x1="38.5" y1="0" x2="3" y2="0" width="0" layer="20"/>
+<wire x1="54.5" y1="3" x2="54.5" y2="1" width="0" layer="20"/>
+<wire x1="54.5" y1="1" x2="55.5" y2="0" width="0" layer="20" curve="90"/>
+<wire x1="55.5" y1="0" x2="91" y2="0" width="0" layer="20"/>
+<wire x1="3" y1="0" x2="37.5" y2="0" width="0" layer="20"/>
+<wire x1="37.5" y1="0" x2="38.5" y2="1" width="0" layer="20" curve="90"/>
+<wire x1="38.5" y1="1" x2="38.5" y2="3" width="0" layer="20"/>
 <wire x1="3" y1="0" x2="0" y2="3" width="0" layer="20" curve="-90"/>
 <wire x1="0" y1="3" x2="0" y2="85" width="0" layer="20"/>
 <wire x1="0" y1="85" x2="3" y2="88" width="0" layer="20" curve="-90"/>
-<wire x1="3" y1="88" x2="91" y2="88" width="0" layer="20"/>
+<wire x1="3" y1="88" x2="61" y2="88" width="0" layer="20"/>
+<wire x1="61" y1="88" x2="62" y2="87" width="0" layer="20" curve="-90"/>
+<wire x1="62" y1="87" x2="62" y2="85" width="0" layer="20"/>
+<wire x1="78" y1="85" x2="78" y2="87" width="0" layer="20"/>
+<wire x1="78" y1="87" x2="79" y2="88" width="0" layer="20" curve="-90"/>
+<wire x1="79" y1="88" x2="91" y2="88" width="0" layer="20"/>
 <wire x1="91" y1="88" x2="94" y2="85" width="0" layer="20" curve="-90"/>
 <wire x1="94" y1="85" x2="94" y2="3" width="0" layer="20"/>
 <wire x1="94" y1="3" x2="91" y2="0" width="0" layer="20" curve="-90"/>
-<wire x1="38.5" y1="0" x2="38.5" y2="3" width="0" layer="20"/>
 <wire x1="38.5" y1="3" x2="41.5" y2="6" width="0" layer="20" curve="-90"/>
 <wire x1="41.5" y1="6" x2="51.5" y2="6" width="0" layer="20"/>
 <wire x1="51.5" y1="6" x2="54.5" y2="3" width="0" layer="20" curve="-90"/>
-<wire x1="54.5" y1="3" x2="54.5" y2="0" width="0" layer="20"/>
 <wire x1="61" y1="57.5" x2="61" y2="13" width="0" layer="20"/>
 <wire x1="61" y1="13" x2="62" y2="12" width="0" layer="20" curve="90"/>
@@
 <rectangle x1="0" y1="0" x2="94" y2="88" layer="29"/>
 <rectangle x1="0" y1="0" x2="94" y2="88" layer="30"/>
+<wire x1="62" y1="85" x2="65" y2="82" width="0" layer="20" curve="90"/>
+<wire x1="65" y1="82" x2="75" y2="82" width="0" layer="20"/>
+<wire x1="75" y1="82" x2="78" y2="85" width="0" layer="20" curve="90"/>
 </plain>
 <attributes>
@@
 <element name="H12" library="OSSI" package="3.2-PAD-ROUND" value="MOUNT-PAD-ROUND3.2" x="9" y="71.5"/>
 <element name="H13" library="OSSI" package="3.2-PAD-ROUND" value="MOUNT-PAD-ROUND3.2" x="9" y="26.5"/>
-<element name="X2" library="OSSI" package="WEIDMULLER1760490000" value="WEIDMULLER" x="68.08" y="80.2"/>
+<element name="X2" library="OSSI" package="WEIDMULLER1760490000" value="WEIDMULLER" x="72.5" y="73.12"/>
 <element name="H14" library="OSSI" package="3.2-PAD-ROUND" value="MOUNT-PAD-ROUND3.2" x="63.5" y="73.12"/>
 <element name="H15" library="OSSI" package="3.2-PAD-ROUND" value="MOUNT-PAD-ROUND3.2" x="63.5" y="63.5"/>
@@
 <polygon width="0.254" layer="16" thermals="no">
 <vertex x="60.325" y="69.85"/>
-<vertex x="67.31" y="69.85"/>
-<vertex x="67.31" y="87.63"/>
-<vertex x="60.325" y="87.63"/>
+<vertex x="71.755" y="69.85"/>
+<vertex x="71.755" y="76.2"/>
+<vertex x="60.325" y="76.2"/>
 </polygon>
 <polygon width="0.254" layer="1" thermals="no">
 <vertex x="60.325" y="69.85"/>
-<vertex x="67.31" y="69.85"/>
-<vertex x="67.31" y="87.63"/>
-<vertex x="60.325" y="87.63"/>
+<vertex x="71.755" y="69.85"/>
+<vertex x="71.755" y="76.2"/>
+<vertex x="60.325" y="76.2"/>
 </polygon>
 </signal>
@@
 <contactref element="H16" pad="B3,2"/>
 <polygon width="0.254" layer="16" thermals="no">
-<vertex x="69.215" y="82.55"/>
-<vertex x="69.215" y="69.85"/>
-<vertex x="71.755" y="69.85"/>
+<vertex x="73.025" y="76.2"/>
+<vertex x="73.025" y="67.31"/>
+<vertex x="71.755" y="67.31"/>
 <vertex x="71.755" y="60.325"/>
 <vertex x="78.105" y="60.325"/>
-<vertex x="78.105" y="82.55"/>
+<vertex x="78.105" y="76.2"/>
 </polygon>
 <polygon width="0.254" layer="1" thermals="no">
-<vertex x="69.215" y="82.55"/>
-<vertex x="69.215" y="69.85"/>
-<vertex x="71.755" y="69.85"/>
+<vertex x="73.025" y="76.2"/>
+<vertex x="73.025" y="67.31"/>
+<vertex x="71.755" y="67.31"/>
 <vertex x="71.755" y="60.325"/>
 <vertex x="78.105" y="60.325"/>
-<vertex x="78.105" y="82.55"/>
-</polygon>
-</signal>
+<vertex x="78.105" y="76.2"/>
+</polygon>
+</signal>
