File: OSSISolarPanel/OSSISolarZ/OSSISolarZ.sch (EAGLE design)
At the start: 41 parts, among them U1 TMP100, U2 MAX4376, X1 DF13DF13A-8P-1.25H

Commit message: New OBC being made
Other:
- note added: "Add Bypass capacitor!!!"
Changed lines of the file:
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@@
 <text x="73.66" y="134.62" size="1.778" layer="94">pull-up resistor needed?</text>
 <text x="114.3" y="116.84" size="1.778" layer="94">power supplied by OBC</text>
+<text x="307.34" y="134.62" size="1.9304" layer="94">Add Bypass capacitor!!!</text>
 </plain>
 <instances>

Commit message: design files are added
Other:
- note added: "configurable address pin"
- note removed: "configurable address pin needs to be added"
- moved on the sheet: C1, D1, D2, D3, D4, D5, D6, D7, D8, H1, H2, H3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
