File: OSSISolarPanel/OSSISolarY/OSSISolarY.sch (EAGLE design)
At the start: 51 parts, among them U1 TMP100, U2 MAX4376, X1 DF13DF13A-8P-1.25H

Commit message: design files are added
Other:
- note added: "configurable address pin"
- note removed: "configurable address pin needs to be added"
- moved on the sheet: C1, D1, D10, D11, D12, D2, D3, D4, D5, D6, D7, D8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
