File: OSSIComms/+XPanelNew/+XPanelNew.brd (EAGLE design)
At the start: 109.5 x 82.5 mm, 19 parts, among them X1 RFCON-MCX-V, X10 P-PAD, X11 P-PAD-S, X2 RFCON-MCX-V, X3 P-PAD-S, X4 P-PAD-S, X5 P-PAD-S, X6 P-PAD, X7 P-PAD, X8 P-PAD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

Commit message: design files are added
Parts:
- L3: value (none) -> 6mm dia, 5 turn
Changed lines of the file:
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@@
 <?xml version="1.0" encoding="utf-8"?>
 <!DOCTYPE eagle SYSTEM "eagle.dtd">
-<eagle version="6.1">
+<eagle version="6.5.0">
 <drawing>
 <settings>
@@
 <layer number="17" name="Pads" color="2" fill="1" visible="yes" active="yes"/>
 <layer number="18" name="Vias" color="2" fill="1" visible="yes" active="yes"/>
-<layer number="19" name="Unrouted" color="6" fill="1" visible="yes" active="yes"/>
+<layer number="19" name="Unrouted" color="6" fill="1" visible="no" active="yes"/>
 <layer number="20" name="Dimension" color="15" fill="1" visible="yes" active="yes"/>
-<layer number="21" name="tPlace" color="7" fill="1" visible="yes" active="yes"/>
-<layer number="22" name="bPlace" color="7" fill="1" visible="yes" active="yes"/>
-<layer number="23" name="tOrigins" color="15" fill="1" visible="yes" active="yes"/>
-<layer number="24" name="bOrigins" color="15" fill="1" visible="yes" active="yes"/>
-<layer number="25" name="tNames" color="7" fill="1" visible="yes" active="yes"/>
-<layer number="26" name="bNames" color="7" fill="1" visible="yes" active="yes"/>
-<layer number="27" name="tValues" color="7" fill="1" visible="yes" active="yes"/>
-<layer number="28" name="bValues" color="7" fill="1" visible="yes" active="yes"/>
+<layer number="21" name="tPlace" color="7" fill="1" visible="no" active="yes"/>
+<layer number="22" name="bPlace" color="7" fill="1" visible="no" active="yes"/>
+<layer number="23" name="tOrigins" color="15" fill="1" visible="no" active="yes"/>
+<layer number="24" name="bOrigins" color="15" fill="1" visible="no" active="yes"/>
+<layer number="25" name="tNames" color="7" fill="1" visible="no" active="yes"/>
+<layer number="26" name="bNames" color="7" fill="1" visible="no" active="yes"/>
+<layer number="27" name="tValues" color="7" fill="1" visible="no" active="yes"/>
+<layer number="28" name="bValues" color="7" fill="1" visible="no" active="yes"/>
 <layer number="29" name="tStop" color="7" fill="3" visible="no" active="yes"/>
 <layer number="30" name="bStop" color="7" fill="6" visible="no" active="yes"/>
@@
 </class>
 </classes>
-<designrules>
+<designrules name="default">
 <description language="de">&lt;b&gt;EAGLE Design Rules&lt;/b&gt;
 &lt;p&gt;
@@
 </autorouter>
 <elements>
-<element name="ADS1" library="OSSI" package="OSSIADS" value="OSSIADS" x="50" y="76.25" rot="R45"/>
-<element name="X1" library="OSSI" package="MCX-V" value="RFCON-MCX-V" x="66.25" y="16" rot="MR0"/>
-<element name="X2" library="OSSI" package="MCX-V" value="RFCON-MCX-V" x="77" y="41.25" rot="MR0"/>
-<element name="LD1" library="OSSI" package="TEMT6000-SEN" value="TEMT6000X01" x="60.5" y="41.25" rot="R90"/>
-<element name="C1" library="OSSI" package="C0805(2012)" value="5.975pF" x="83" y="41.25" rot="MR0"/>
-<element name="L1" library="OSSI" package="L0805(2012)" value="22.4nH" x="83" y="39.25" rot="MR180"/>
-<element name="L2" library="OSSI" package="L0805(2012)" value="22.4nH" x="83.75" y="43.75" rot="MR0"/>
-<element name="C2" library="OSSI" package="C0805(2012)" value="5.975pF" x="83.75" y="37" rot="MR0"/>
-<element name="R1" library="OSSI" package="R0805(2012)" value="10k" x="63.5" y="40.5" rot="MR270"/>
-<element name="X3" library="OSSI" package="P-PAD-S" value="P-PAD-S" x="66.25" y="47.75" rot="MR270"/>
-<element name="X4" library="OSSI" package="P-PAD-S" value="P-PAD-S" x="63.5" y="47.75" rot="MR270"/>
-<element name="X5" library="OSSI" package="P-PAD-S" value="P-PAD-S" x="60.5" y="47.75" rot="MR270"/>
-<element name="X6" library="OSSI" package="P-PAD" value="P-PAD" x="50" y="3.25"/>
-<element name="X7" library="OSSI" package="P-PAD" value="P-PAD" x="85" y="50.750003125" rot="R270"/>
-<element name="X8" library="OSSI" package="P-PAD" value="P-PAD" x="85" y="31.75" rot="R90"/>
-<element name="X9" library="OSSI" package="P-PAD" value="P-PAD" x="51.25" y="69.5" rot="MR0"/>
-<element name="X10" library="OSSI" package="P-PAD" value="P-PAD" x="54.75" y="66" rot="MR0"/>
-<element name="L3" library="rcl" package="0207/10" value="" x="55" y="11" rot="MR180"/>
-<element name="X11" library="OSSI" package="P-PAD-S" value="P-PAD-S" x="61" y="16" rot="MR0"/>
+<element name="ADS1" library="OSSI" package="OSSIADS" value="OSSIADS" x="50" y="76.25" smashed="yes" rot="R45">
+<attribute name="NAME" x="66.164459375" y="75.2894875" size="1.27" layer="25" font="vector" rot="R45"/>
+<attribute name="VALUE" x="67.960509375" y="56.493434375" size="1.778" layer="27" rot="R45"/>
+</element>
+<element name="X1" library="OSSI" package="MCX-V" value="RFCON-MCX-V" x="66.25" y="16" smashed="yes" rot="MR0">
+<attribute name="NAME" x="66.79" y="20.445" size="1.27" layer="26" font="vector" rot="MR0"/>
+<attribute name="VALUE" x="69.425" y="10.285" size="1.27" layer="28" rot="MR0"/>
+</element>
+<element name="X2" library="OSSI" package="MCX-V" value="RFCON-MCX-V" x="77" y="41.25" smashed="yes" rot="MR0">
+<attribute name="NAME" x="72.54" y="40.695" size="1.27" layer="26" font="vector" rot="MR0"/>
+<attribute name="VALUE" x="80.175" y="35.535" size="1.27" layer="28" rot="MR0"/>
+</element>
+<element name="LD1" library="OSSI" package="TEMT6000-SEN" value="TEMT6000X01" x="60.5" y="41.25" smashed="yes" rot="R90">
+<attribute name="NAME" x="59.119" y="40.234" size="1.27" layer="25" font="vector" rot="R90"/>
+<attribute name="VALUE" x="61.262" y="40.234" size="0.4064" layer="27" rot="R90"/>
+</element>
+<element name="C1" library="OSSI" package="C0805(2012)" value="5.975pF" x="83" y="41.25" smashed="yes" rot="MR0">
+<attribute name="NAME" x="86.889" y="40.766" size="1.27" layer="26" font="vector" rot="MR0"/>
+<attribute name="VALUE" x="83.889" y="38.964" size="1.27" layer="28" rot="MR0"/>
+</element>
+<element name="L1" library="OSSI" package="L0805(2012)" value="22.4nH" x="83" y="39.25" smashed="yes" rot="MR180">
+<attribute name="NAME" x="84.611" y="39.734" size="1.27" layer="26" font="vector" rot="MR180"/>
+<attribute name="VALUE" x="82.111" y="41.536" size="1.27" layer="28" rot="MR180"/>
+</element>
+<element name="L2" library="OSSI" package="L0805(2012)" value="22.4nH" x="83.75" y="43.75" smashed="yes" rot="MR0">
+<attribute name="NAME" x="87.639" y="43.266" size="1.27" layer="26" font="vector" rot="MR0"/>
+<attribute name="VALUE" x="84.639" y="41.464" size="1.27" layer="28" rot="MR0"/>
+</element>
+<element name="C2" library="OSSI" package="C0805(2012)" value="5.975pF" x="83.75" y="37" smashed="yes" rot="MR0">
+<attribute name="NAME" x="87.639" y="36.516" size="1.27" layer="26" font="vector" rot="MR0"/>
+<attribute name="VALUE" x="84.639" y="34.714" size="1.27" layer="28" rot="MR0"/>
+</element>
+<element name="R1" library="OSSI" package="R0805(2012)" value="10k" x="63.5" y="40.5" smashed="yes" rot="MR270">
+<attribute name="NAME" x="66.484" y="42.389" size="1.27" layer="26" font="vector" rot="MR270"/>
+<attribute name="VALUE" x="65.786" y="41.389" size="1.27" layer="28" rot="MR270"/>
+</element>
+<element name="X3" library="OSSI" package="P-PAD-S" value="P-PAD-S" x="66.25" y="47.75" smashed="yes" rot="MR270">
+<attribute name="NAME" x="66.98" y="53.29" size="1.27" layer="26" font="vector" rot="MR270"/>
+<attribute name="VALUE" x="68.79" y="50.29" size="1.27" layer="28" rot="MR270"/>
+</element>
+<element name="X4" library="OSSI" package="P-PAD-S" value="P-PAD-S" x="63.5" y="47.75" smashed="yes" rot="MR270">
+<attribute name="NAME" x="64.23" y="53.29" size="1.27" layer="26" font="vector" rot="MR270"/>
+<attribute name="VALUE" x="66.04" y="50.29" size="1.27" layer="28" rot="MR270"/>
+</element>
+<element name="X5" library="OSSI" package="P-PAD-S" value="P-PAD-S" x="60.5" y="47.75" smashed="yes" rot="MR270">
+<attribute name="NAME" x="61.23" y="53.29" size="1.27" layer="26" font="vector" rot="MR270"/>
+<attribute name="VALUE" x="63.04" y="50.29" size="1.27" layer="28" rot="MR270"/>
+</element>
+<element name="X6" library="OSSI" package="P-PAD" value="P-PAD" x="50" y="3.25" smashed="yes">
+<attribute name="NAME" x="54.19" y="2.52" size="1.27" layer="25" font="vector"/>
+<attribute name="VALUE" x="46.19" y="0.71" size="1.27" layer="27"/>
+</element>
+<element name="X7" library="OSSI" package="P-PAD" value="P-PAD" x="85" y="50.750003125" smashed="yes" rot="R270">
+<attribute name="NAME" x="86.27" y="51.560003125" size="1.27" layer="25" font="vector" rot="R270"/>
+<attribute name="VALUE" x="82.46" y="54.560003125" size="1.27" layer="27" rot="R270"/>
+</element>
+<element name="X8" library="OSSI" package="P-PAD" value="P-PAD" x="85" y="31.75" smashed="yes" rot="R90">
+<attribute name="NAME" x="87.73" y="30.94" size="1.27" layer="25" font="vector" rot="R90"/>
+<attribute name="VALUE" x="87.54" y="27.94" size="1.27" layer="27" rot="R90"/>
+</element>
+<element name="X9" library="OSSI" package="P-PAD" value="P-PAD" x="51.25" y="69.5" smashed="yes" rot="MR0">
+<attribute name="NAME" x="50.06" y="70.77" size="1.27" layer="26" font="vector" rot="MR0"/>
+<attribute name="VALUE" x="55.06" y="66.96" size="1.27" layer="28" rot="MR0"/>
+</element>
+<element name="X10" library="OSSI" package="P-PAD" value="P-PAD" x="54.75" y="66" smashed="yes" rot="MR0">
+<attribute name="NAME" x="51.56" y="65.27" size="1.27" layer="26" font="vector" rot="MR0"/>
+<attribute name="VALUE" x="58.56" y="63.46" size="1.27" layer="28" rot="MR0"/>
+</element>
+<element name="L3" library="rcl" package="0207/10" value="6mm dia, 5 turn" x="55" y="11" smashed="yes" rot="MR180">
+<attribute name="NAME" x="53.952" y="13.476" size="1.27" layer="26" font="vector" rot="MR180"/>
+<attribute name="VALUE" x="52.7394" y="11.635" size="1.27" layer="28" ratio="10" rot="MR180"/>
+</element>
+<element name="X11" library="OSSI" package="P-PAD-S" value="P-PAD-S" x="61" y="16" smashed="yes" rot="MR0">
+<attribute name="NAME" x="58.54" y="15.27" size="1.27" layer="26" font="vector" rot="MR0"/>
+<attribute name="VALUE" x="63.54" y="13.46" size="1.27" layer="28" rot="MR0"/>
+</element>
 </elements>
 <signals>
