File: OSSIComms/+XPanelNew/+XPanelNew.sch (EAGLE design)
At the start: 19 parts, among them X1 RFCON-MCX-V, X10 P-PAD, X11 P-PAD-S, X2 RFCON-MCX-V, X3 P-PAD-S, X4 P-PAD-S, X5 P-PAD-S, X6 P-PAD, X7 P-PAD, X8 P-PAD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

Commit message: front panel value
Other:
- note added: "0603HC_22NX coilcraft is used"
- note added: "6pF is used"
Changed lines of the file:
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@@
 <text x="172.72" y="114.3" size="1.778" layer="94">LC Balun</text>
 <text x="121.92" y="58.42" size="5.08" layer="94">MOVE INDUCTOR TO AVOID COLLISION!!!!!!</text>
+<text x="154.94" y="116.84" size="1.778" layer="94">0603HC_22NX coilcraft is used</text>
+<text x="152.4" y="147.32" size="1.778" layer="94">6pF is used</text>
 </plain>
 <instances>

Commit message: design files are added
Parts:
- L3: value (none) -> 6mm dia, 5 turn
Other:
- note added: "12pF cap connected to 1 turn from X6 and Ground"
- note added: "Antenna Deployment System"
- note added: "Connect 12pF ceramic Cap from the L3 to GND"
- note added: "UHF"
- note added: "VHF"
- note removed: "MOVE INDUCTOR TO AVOID COLLISION!!!!!!"
- moved on the sheet: ADS1, C1, C2, L1, L2, L3, LD1, R1, X1, X10, X11, X2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
